Commit message: Change the order of wheels

File: living_lab_robot_description/urdf/mobile_assy.urdf.xacro (robot description, xacro)
@@ -85,4 +85,30 @@
     </joint>
     <xacro:insert_velocity_transmission name="omni_wheel_1_joint" />
+    <link name="omni_wheel_3">
+        <visual>
+            <origin xyz="0 0 0" rpy="0 0 0"/>
+            <geometry>
+                <mesh filename="package://living_lab_robot_description/meshes/omni_wheel.dae" scale="1 1 1"/>
+            </geometry>
+        </visual>
+        <collision>
+            <origin xyz="0 0 0" rpy="0 0 0"/>
+            <geometry>
+                <mesh filename="package://living_lab_robot_description/meshes/omni_wheel.dae" scale="1 1 1"/>
+            </geometry>
+        </collision>
+        <inertial>
+            <origin xyz="0 0 0" rpy="0 0 0"/>
+            <mass value="1.0"/>
+            <inertia ixx="1.0" ixy="0.0" ixz="0.0" iyy="1.0" iyz="0.0" izz="1.0"/>
+        </inertial>
+    </link>
+    <joint name="omni_wheel_3_joint" type="continuous">
+        <parent link="base_link"/>
+        <child link="omni_wheel_3"/>
+        <origin xyz="${0.282 * cos(pi/3)}  ${0.282 * sin(-pi/3)} 0" rpy="0 0 ${-5*pi/6}"/>
+        <axis xyz="0 1 0"/>
+    </joint>
+    <xacro:insert_velocity_transmission name="omni_wheel_3_joint" />
     <link name="omni_wheel_2">
         <visual>
@@ -107,33 +133,7 @@
         <parent link="base_link"/>
         <child link="omni_wheel_2"/>
-        <origin xyz="${0.282 * cos(pi/3)}  ${0.282 * sin(-pi/3)} 0" rpy="0 0 ${-5*pi/6}"/>
+        <origin xyz="-0.282 0 0" rpy="0 0 ${pi/2}"/>
         <axis xyz="0 1 0"/>
     </joint>
     <xacro:insert_velocity_transmission name="omni_wheel_2_joint" />
-    <link name="omni_wheel_3">
-        <visual>
-            <origin xyz="0 0 0" rpy="0 0 0"/>
-            <geometry>
-                <mesh filename="package://living_lab_robot_description/meshes/omni_wheel.dae" scale="1 1 1"/>
-            </geometry>
-        </visual>
-        <collision>
-            <origin xyz="0 0 0" rpy="0 0 0"/>
-            <geometry>
-                <mesh filename="package://living_lab_robot_description/meshes/omni_wheel.dae" scale="1 1 1"/>
-            </geometry>
-        </collision>
-        <inertial>
-            <origin xyz="0 0 0" rpy="0 0 0"/>
-            <mass value="1.0"/>
-            <inertia ixx="1.0" ixy="0.0" ixz="0.0" iyy="1.0" iyz="0.0" izz="1.0"/>
-        </inertial>
-    </link>
-    <joint name="omni_wheel_3_joint" type="continuous">
-        <parent link="base_link"/>
-        <child link="omni_wheel_3"/>
-        <origin xyz="-0.282 0 0" rpy="0 0 ${pi/2}"/>
-        <axis xyz="0 1 0"/>
-    </joint>
-    <xacro:insert_velocity_transmission name="omni_wheel_3_joint" />
 </robot>
