Commit message: Remodeling for C3
Modified collada files

Edit moveit_config

File: living_lab_robot_description/urdf/gazebo.urdf.xacro (robot description, xacro)
@@ -16,39 +16,41 @@
         </plugin>
     </gazebo>
-    <gazebo reference="hokuyo_link">
-        <sensor type="ray" name="hokuyo_sensor">
-            <pose>0 0 0 0 0 0</pose>
-            <visualize>true</visualize>
-            <update_rate>40</update_rate>
-            <ray>
-                <scan>
-                    <horizontal>
-                        <samples>720</samples>
-                        <resolution>1</resolution>
-                        <min_angle>-1.66</min_angle>
-                        <max_angle>1.66</max_angle>
-                    </horizontal>
-                </scan>
-                <range>
-                    <min>0.10</min>
-                    <max>30.0</max>
-                    <resolution>0.01</resolution>
-                </range>
-                <noise>
-                    <type>gaussian</type>
-                    <!-- Noise parameters based on published spec for Hokuyo laser
-                         achieving "+-30mm" accuracy at range < 10m.  A mean of 0.0m and
-                         stddev of 0.01m will put 99.7% of samples within 0.03m of the true
-                         reading. -->
-                    <mean>0.0</mean>
-                    <stddev>0.01</stddev>
-                </noise>
-            </ray>
-            <plugin name="gazebo_hokuyo_controller" filename="libgazebo_ros_laser.so">
-                <topicName>scan</topicName>
-                <frameName>hokuyo_link</frameName>
-            </plugin>
-        </sensor>
-  </gazebo>
+    <xacro:macro name="insert_hokuyo_sensor" params="name">
+        <gazebo reference="${name}_hokuyo_link">
+            <sensor type="ray" name="${name}_hokuyo_sensor">
+                <pose>0 0 0 0 0 0</pose>
+                <visualize>false</visualize>
+                <update_rate>30</update_rate>
+                <ray>
+                    <scan>
+                        <horizontal>
+                            <samples>720</samples>
+                            <resolution>1</resolution>
+                            <min_angle>-1.6</min_angle>
+                            <max_angle>1.6</max_angle>
+                        </horizontal>
+                    </scan>
+                    <range>
+                        <min>0.10</min>
+                        <max>30.0</max>
+                        <resolution>0.01</resolution>
+                    </range>
+                    <noise>
+                        <type>gaussian</type>
+                        <!-- Noise parameters based on published spec for Hokuyo laser
+                            achieving "+-30mm" accuracy at range < 10m.  A mean of 0.0m and
+                            stddev of 0.01m will put 99.7% of samples within 0.03m of the true
+                            reading. -->
+                        <mean>0.0</mean>
+                        <stddev>0.01</stddev>
+                    </noise>
+                </ray>
+                <plugin name="gazebo_hokuyo_controller" filename="libgazebo_ros_laser.so">
+                    <topicName>${name}/scan</topicName>
+                    <frameName>${name}_hokuyo_link</frameName>
+                </plugin>
+            </sensor>
+        </gazebo>
+    </xacro:macro>
     <xacro:macro name="insert_camera_sensor" params="name">
         <gazebo reference="${name}">

File: living_lab_robot_description/urdf/robot.urdf.xacro (robot description, xacro)
@@ -3,342 +3,9 @@
     <xacro:include filename="$(find living_lab_robot_description)/urdf/gazebo.urdf.xacro"/>
     <xacro:include filename="$(find living_lab_robot_description)/urdf/transmission.urdf.xacro"/>
-    <link name="base_footprint">
-        <visual>
-            <origin xyz="0 0 0" rpy="0 0 0" />
-            <geometry>
-                <box size="0.001 0.001 0.001" />
-            </geometry>
-        </visual>
-    </link>
-    <link name="base_link">
-        <visual>
-            <origin xyz="0 0 0" rpy="0 0 0"/>
-            <geometry>
-                <mesh filename="package://living_lab_robot_description/meshes/omni_base.dae" scale="1 1 1"/>
-            </geometry>
-        </visual>
-        <collision>
-            <origin xyz="0 0 0" rpy="0 0 0"/>
-            <geometry>
-                <mesh filename="package://living_lab_robot_description/meshes/omni_base.dae" scale="1 1 1"/>
-            </geometry>
-        </collision>
-        <inertial>
-            <origin xyz="0 0 0" rpy="0 0 0"/>
-            <mass value="30.0"/>
-            <inertia ixx="1.0" ixy="0.0" ixz="0.0" iyy="1.0" iyz="0.0" izz="1.0"/>
-        </inertial>
-    </link>
-    <joint name="base_link_joint" type="fixed">
-        <parent link="base_footprint"/>
-        <child link="base_link"/>
-        <origin xyz="0 0 0.095" rpy="0 0 0"/>
-    </joint>
-    <link name="elv_base_link">
-        <visual>
-            <origin xyz="0 0 0" rpy="0 0 0"/>
-            <geometry>
-                <mesh filename="package://living_lab_robot_description/meshes/elv_base.dae" scale="1 1 1"/>
-            </geometry>
-        </visual>
-        <collision>
-            <origin xyz="0 0 0" rpy="0 0 0"/>
-            <geometry>
-                <mesh filename="package://living_lab_robot_description/meshes/elv_base.dae" scale="1 1 1"/>
-            </geometry>
-        </collision>
-        <inertial>
-            <origin xyz="0 0 0" rpy="0 0 0"/>
-            <mass value="1.0"/>
-            <inertia ixx="1.0" ixy="0.0" ixz="0.0" iyy="1.0" iyz="0.0" izz="1.0"/>
-        </inertial>
-    </link>
-    <joint name="elv_base_rotate_joint" type="revolute">
-        <parent link="base_link"/>
-        <child link="elv_base_link"/>
-        <origin xyz="0 0 0.21" rpy="0 0 0"/>
-        <axis xyz="0 0 1"/>
-        <limit lower="${-90/180*pi}" upper="${90/180*pi}" velocity="1.0" effort="1000"/>
-    </joint>
-    <xacro:insert_position_transmission name="elv_base_rotate_joint" />
-    <link name="elv_mount_link">
-        <visual>
-            <origin xyz="0 0 -0.07" rpy="0 ${pi/2} 0"/>
-            <geometry>
-                <mesh filename="package://living_lab_robot_description/meshes/elv_mount.dae" scale="1 1 1"/>
-            </geometry>
-        </visual>
-        <collision>
-            <origin xyz="0 0 0" rpy="0 ${pi/2} 0"/>
-            <geometry>
-                <mesh filename="package://living_lab_robot_description/meshes/elv_mount.dae" scale="1 1 1"/>
-            </geometry>
-        </collision>
-        <inertial>
-            <origin xyz="0 0 0" rpy="0 0 0"/>
-            <mass value="1.0"/>
-            <inertia ixx="1.0" ixy="0.0" ixz="0.0" iyy="1.0" iyz="0.0" izz="1.0"/>
-        </inertial>
-    </link>
-    <joint name="elv_base_trans_joint" type="prismatic">
-        <parent link="elv_base_link"/>
-        <child link="elv_mount_link"/>
-        <origin xyz="0.01 0 0.6865" rpy="0 0 0"/>
-        <axis xyz="0 0 1"/>
-        <limit lower="-0.5" upper="0.0" velocity="1.0" effort="1000"/>
-    </joint>
-    <xacro:insert_position_transmission name="elv_base_trans_joint" />
-    <link name="projector_pan">
-        <visual>
-            <origin xyz="0 0 0" rpy="0 0 0"/>
-            <geometry>
-                <mesh filename="package://living_lab_robot_description/meshes/proj_pan.dae" scale="1 1 1"/>
-            </geometry>
-        </visual>
-        <collision>
-            <origin xyz="0 0 0" rpy="0 0 0"/>
-            <geometry>
-                <mesh filename="package://living_lab_robot_description/meshes/proj_pan.dae" scale="1 1 1"/>
-            </geometry>
-        </collision>
-        <inertial>
-            <origin xyz="0 0 0" rpy="0 0 0"/>
-            <mass value="1.0"/>
-            <inertia ixx="1.0" ixy="0.0" ixz="0.0" iyy="1.0" iyz="0.0" izz="1.0"/>
-        </inertial>
-    </link>
-    <joint name="projector_pan_joint" type="revolute">
-        <parent link="elv_base_link"/>
-        <child link="projector_pan"/>
-        <origin xyz="-0.025 0 0.71" rpy="0 0 0"/>
-        <axis xyz="0 0 1"/>
-        <limit lower="${-90/180*pi}" upper="${90/180*pi}" velocity="1.0" effort="1000"/>
-    </joint>
-    <xacro:insert_position_transmission name="projector_pan_joint" />
-    <link name="projector_tilt">
-        <visual>
-            <origin xyz="0 0 0" rpy="0 0 0"/>
-            <geometry>
-                <mesh filename="package://living_lab_robot_description/meshes/proj_tilt.dae" scale="1 1 1"/>
-            </geometry>
-        </visual>
-        <collision>
-            <origin xyz="0 0 0" rpy="0 0 0"/>
-            <geometry>
-                <mesh filename="package://living_lab_robot_description/meshes/proj_tilt.dae" scale="1 1 1"/>
-            </geometry>
-        </collision>
-        <inertial>
-            <origin xyz="0 0 0" rpy="0 0 0"/>
-            <mass value="1.0"/>
-            <inertia ixx="1.0" ixy="0.0" ixz="0.0" iyy="1.0" iyz="0.0" izz="1.0"/>
-        </inertial>
-    </link>
-    <joint name="projector_tilt_joint" type="revolute">
-        <parent link="projector_pan"/>
-        <child link="projector_tilt"/>
-        <origin xyz="0 0 0.0785" rpy="0 0 0"/>
-        <axis xyz="0 1 0"/>
-        <limit lower="${-90/180*pi}" upper="${90/180*pi}" velocity="1.0" effort="1000"/>
-    </joint>
-    <xacro:insert_position_transmission name="projector_tilt_joint" />
-    <link name="arm_link1">
-        <visual>
-            <origin xyz="0.09 0 0" rpy="0 ${pi/2} 0"/>
-            <geometry>
-                <mesh filename="package://living_lab_robot_description/meshes/arm_link1.stl" scale="0.001 0.001 0.001"/>
-            </geometry>
-        </visual>
-        <collision>
-            <origin xyz="0.09 0 0" rpy="0 0 0"/>
-            <geometry>
-                <mesh filename="package://living_lab_robot_description/meshes/arm_link1.stl" scale="0.001 0.001 0.001"/>
-            </geometry>
-        </collision>
-        <inertial>
-            <origin xyz="0 0 0" rpy="0 0 0"/>
-            <mass value="1.0"/>
-            <inertia ixx="1.0" ixy="0.0" ixz="0.0" iyy="1.0" iyz="0.0" izz="1.0"/>
-        </inertial>
-    </link>
-    <joint name="arm_fixed_base" type="fixed">
-        <parent link="elv_mount_link"/>
-        <child link="arm_link1"/>
-        <origin xyz="0.01 0 -0.03" rpy="0 0 0"/>
-    </joint>
-    <link name="arm_link2">
-        <visual>
-            <origin xyz="-0.036 0 0" rpy="${-pi/2} 0 ${-pi/2}"/>
-            <geometry>
-                <mesh filename="package://living_lab_robot_description/meshes/arm_link2.dae" scale="1 1 1"/>
-            </geometry>
-        </visual>
-        <collision>
-            <origin xyz="0 0 0" rpy="0 0 0"/>
-            <geometry>
-                <mesh filename="package://living_lab_robot_description/meshes/arm_link2.dae" scale="1 1 1"/>
-            </geometry>
-        </collision>
-        <inertial>
-            <origin xyz="0 0 0" rpy="0 0 0"/>
-            <mass value="1.0"/>
-            <inertia ixx="1.0" ixy="0.0" ixz="0.0" iyy="1.0" iyz="0.0" izz="1.0"/>
-        </inertial>
-    </link>
-    <joint name="arm_joint1" type="revolute">
-        <parent link="arm_link1"/>
-        <child link="arm_link2"/>
-        <origin xyz="0.128 0 0" rpy="0 0 0"/>
-         <axis xyz="1 0 0"/>
-        <limit lower="${-90/180*pi}" upper="${90/180*pi}" velocity="1.0" effort="1000"/>
-    </joint>
-    <xacro:insert_position_transmission name="arm_joint1" />
-    <link name="arm_link3">
-        <visual>
-            <origin xyz="-0.069 0 0" rpy="${-pi/2} 0 ${-pi/2}"/>
-            <geometry>
-                <mesh filename="package://living_lab_robot_description/meshes/arm_link3.dae" scale="1 1 1"/>
-            </geometry>
-        </visual>
-        <collision>
-            <origin xyz="0 0 0" rpy="0 0 0"/>
-            <geometry>
-                <mesh filename="package://living_lab_robot_description/meshes/arm_link3.dae" scale="1 1 1"/>
-            </geometry>
-        </collision>
-        <inertial>
-            <origin xyz="0 0 0" rpy="0 0 0"/>
-            <mass value="1.0"/>
-            <inertia ixx="1.0" ixy="0.0" ixz="0.0" iyy="1.0" iyz="0.0" izz="1.0"/>
-        </inertial>
-    </link>
-    <joint name="arm_joint2" type="revolute">
-        <parent link="arm_link2"/>
-        <child link="arm_link3"/>
-        <origin xyz="0.033 0 0" rpy="0 0 0"/>
-         <axis xyz="0 1 0"/>
-        <limit lower="${-90/180*pi}" upper="${90/180*pi}" velocity="1.0" effort="1000"/>
-    </joint>
-    <xacro:insert_position_transmission name="arm_joint2" />
-    <link name="arm_link4">
-        <visual>
-            <origin xyz="0 0 0" rpy="0 0 0"/>
-            <geometry>
-                <mesh filename="package://living_lab_robot_description/meshes/arm_link4.dae" scale="1 1 1"/>
-            </geometry>
-        </visual>
-        <collision>
-            <origin xyz="0 0 0" rpy="0 0 0"/>
-            <geometry>
-                <mesh filename="package://living_lab_robot_description/meshes/arm_link4.dae" scale="1 1 1"/>
-            </geometry>
-        </collision>
-        <inertial>
-            <origin xyz="0 0 0" rpy="0 0 0"/>
-            <mass value="1.0"/>
-            <inertia ixx="1.0" ixy="0.0" ixz="0.0" iyy="1.0" iyz="0.0" izz="1.0"/>
-        </inertial>
-    </link>
-    <joint name="arm_joint3" type="revolute">
-        <parent link="arm_link3"/>
-        <child link="arm_link4"/>
-        <origin xyz="0.264 0 0.03" rpy="0 0 0"/>
-        <axis xyz="0 1 0"/>
-        <limit lower="${-90/180*pi}" upper="${90/180*pi}" velocity="1.0" effort="1000"/>
-    </joint>
-    <xacro:insert_position_transmission name="arm_joint3" />
-    <link name="arm_link5">
-        <visual>
-            <origin xyz="0 0 0" rpy="0 0 0"/>
-            <geometry>
-                <mesh filename="package://living_lab_robot_description/meshes/arm_link5.dae" scale="1 1 1"/>
-            </geometry>
-        </visual>
-        <collision>
-            <origin xyz="0 0 0" rpy="0 0 0"/>
-            <geometry>
-                <mesh filename="package://living_lab_robot_description/meshes/arm_link5.dae" scale="1 1 1"/>
-            </geometry>
-        </collision>
-        <inertial>
-            <origin xyz="0 0 0" rpy="0 0 0"/>
-            <mass value="1.0"/>
-            <inertia ixx="1.0" ixy="0.0" ixz="0.0" iyy="1.0" iyz="0.0" izz="1.0"/>
-        </inertial>
-    </link>
-    <joint name="arm_joint4" type="revolute">
-        <parent link="arm_link4"/>
-        <child link="arm_link5"/>
-        <origin xyz="0.03 0 0.286" rpy="0 0 0"/>
-        <axis xyz="0 0 1"/>
-        <limit lower="${-90/180*pi}" upper="${90/180*pi}" velocity="1.0" effort="1000"/>
-    </joint>
-    <xacro:insert_position_transmission name="arm_joint4" />
-    <link name="arm_link6">
-        <visual>
-            <origin xyz="0 0 0" rpy="0 0 0"/>
-            <geometry>
-                <mesh filename="package://living_lab_robot_description/meshes/arm_link6.dae" scale="1 1 1"/>
-            </geometry>
-        </visual>
-        <collision>
-            <origin xyz="0 0 0" rpy="0 0 0"/>
-            <geometry>
-                <mesh filename="package://living_lab_robot_description/meshes/arm_link6.dae" scale="1 1 1"/>
-            </geometry>
-        </collision>
-        <inertial>
-            <origin xyz="0 0 0" rpy="0 0 0"/>
-            <mass value="1.0"/>
-            <inertia ixx="1.0" ixy="0.0" ixz="0.0" iyy="1.0" iyz="0.0" izz="1.0"/>
-        </inertial>
-    </link>
-    <joint name="arm_joint5" type="revolute">
-        <parent link="arm_link5"/>
-        <child link="arm_link6"/>
-        <origin xyz="0 0 0.035" rpy="0 0 0"/>
-        <axis xyz="0 1 0"/>
-        <limit lower="${-90/180*pi}" upper="${90/180*pi}" velocity="1.0" effort="1000"/>
-    </joint>
-    <xacro:insert_position_transmission name="arm_joint5" />
-    <link name="end_effector">
-        <inertial>
-            <origin xyz="0 0 0" rpy="0 0 0"/>
-            <mass value="0.1"/>
-            <inertia ixx="1.0" ixy="0.0" ixz="0.0" iyy="1.0" iyz="0.0" izz="1.0"/>
-        </inertial>
-    </link>
-    <joint name="end_effector_joint" type="revolute">
-        <parent link="arm_link6"/>
-        <child link="end_effector"/>
-        <origin xyz="0 0 0.124" rpy="0 0 0"/>
-        <axis xyz="0 0 1"/>
-        <limit lower="${-90/180*pi}" upper="${90/180*pi}" velocity="1.0" effort="1000"/>
-    </joint>
-    <xacro:insert_position_transmission name="end_effector_joint" />
-    <!-- Laser Scanner -->
-    <link name="hokuyo_link">
-        <visual>
-            <origin xyz="-0.04 0.03 -0.05" rpy="0 0 0"/>
-            <geometry>
-                <mesh filename="package://living_lab_robot_description/meshes/hokuyo.dae" scale="1 1 1"/>
-            </geometry>
-        </visual>
-        <collision>
-            <origin xyz="0 0 0" rpy="0 0 0"/>
-            <geometry>
-                <mesh filename="package://living_lab_robot_description/meshes/hokuyo.dae" scale="1 1 1"/>
-            </geometry>
-        </collision>
-        <inertial>
-            <origin xyz="0 0 0" rpy="0 0 0"/>
-            <mass value="1.0"/>
-            <inertia ixx="1.0" ixy="0.0" ixz="0.0" iyy="1.0" iyz="0.0" izz="1.0"/>
-        </inertial>
-    </link>
-    <joint name="hokuyo_mount_joint" type="fixed">
-        <parent link="base_link"/>
-        <child link="hokuyo_link"/>
-        <origin xyz="0.21 0 0.15" rpy="0 0 0"/>
-    </joint>
+    <xacro:include filename="$(find living_lab_robot_description)/urdf/mobile_assy.urdf.xacro"/>
+    <xacro:include filename="$(find living_lab_robot_description)/urdf/body_assy.urdf.xacro"/>
+    <xacro:include filename="$(find living_lab_robot_description)/urdf/robotis_arm.urdf.xacro"/>
+    <xacro:include filename="$(find living_lab_robot_description)/urdf/robotis_gripper.urdf.xacro"/>
+    <xacro:include filename="$(find living_lab_robot_description)/urdf/head1_assy.urdf.xacro"/>
+    <xacro:include filename="$(find living_lab_robot_description)/urdf/head2_assy.urdf.xacro"/>
 </robot>

Commit message: Attach RGBD camera for gazebo

File: living_lab_robot_description/urdf/gazebo.urdf.xacro (robot description, xacro)
@@ -94,3 +94,41 @@
         </gazebo>
     </xacro:macro>
+    <xacro:macro name="insert_rgbd_camera_sensor" params="name">
+        <gazebo reference="${name}_link">
+            <sensor type="depth" name="${name}">
+                <always_on>true</always_on>
+                <update_rate>30.0</update_rate>
+                <camera>
+                    <horizontal_fov>${60.0*pi/180.0}</horizontal_fov>
+                    <image>
+                        <format>R8G8B8</format>
+                        <width>640</width>
+                        <height>480</height>
+                    </image>
+                    <clip>
+                        <near>0.05</near>
+                        <far>8.0</far>
+                    </clip>
+                </camera>
+                <plugin name="kinect_camera_controller" filename="libgazebo_ros_openni_kinect.so">
+                    <cameraName>${name}</cameraName>
+                    <alwaysOn>true</alwaysOn>
+                    <updateRate>30</updateRate>
+                    <imageTopicName>rgb/image_raw</imageTopicName>
+                    <depthImageTopicName>depth_registered/image_raw</depthImageTopicName>
+                    <pointCloudTopicName>depth_registered/points</pointCloudTopicName>
+                    <cameraInfoTopicName>rgb/camera_info</cameraInfoTopicName>
+                    <depthImageCameraInfoTopicName>depth_registered/camera_info</depthImageCameraInfoTopicName>
+                    <frameName>${name}_depth_optical_frame</frameName>
+                    <baseline>0.1</baseline>
+                    <distortion_k1>0.0</distortion_k1>
+                    <distortion_k2>0.0</distortion_k2>
+                    <distortion_k3>0.0</distortion_k3>
+                    <distortion_t1>0.0</distortion_t1>
+                    <distortion_t2>0.0</distortion_t2>
+                    <pointCloudCutoff>0.4</pointCloudCutoff>
+                </plugin>
+            </sensor>
+        </gazebo>
+    </xacro:macro>
 </robot>

File: living_lab_robot_description/urdf/head2_assy.urdf.xacro (robot description, xacro)
@@ -47,4 +47,5 @@
         </inertial>
     </link>
+    <xacro:insert_rgbd_camera_sensor name="head2_d435"/>
     <joint name="head2_d435_tilt_joint" type="revolute">
         <parent link="head2_assy"/>

File: living_lab_robot_description/urdf/mobile_assy.urdf.xacro (robot description, xacro)
@@ -24,6 +24,6 @@
         <inertial>
             <origin xyz="0 0 0" rpy="0 0 0"/>
-            <mass value="30.0"/>
-            <inertia ixx="1.0" ixy="0.0" ixz="0.0" iyy="1.0" iyz="0.0" izz="1.0"/>
+            <mass value="1.0"/>
+            <inertia ixx="10.0" ixy="0.0" ixz="0.0" iyy="10.0" iyz="0.0" izz="10.0"/>
         </inertial>
     </link>

Commit message: Bug fixed

File: living_lab_robot_description/urdf/gazebo.urdf.xacro (robot description, xacro)
@@ -31,10 +31,10 @@
                             <samples>720</samples>
                             <resolution>1</resolution>
-                            <min_angle>-1.6</min_angle>
-                            <max_angle>1.6</max_angle>
+                            <min_angle>-1.5707</min_angle>
+                            <max_angle>1.5707</max_angle>
                         </horizontal>
                     </scan>
                     <range>
-                        <min>0.10</min>
+                        <min>0.15</min>
                         <max>30.0</max>
                         <resolution>0.01</resolution>

File: living_lab_robot_description/urdf/mobile_assy.urdf.xacro (robot description, xacro)
@@ -37,5 +37,5 @@
         <parent link="base_link"/>
         <child link="front_hokuyo_link"/>
-        <origin xyz="0.27 0 0.175" rpy="0 0 0"/>
+        <origin xyz="0.27 0 0.165" rpy="0 0 0"/>
     </joint>
     <link name="rear_hokuyo_link">
@@ -50,5 +50,5 @@
         <parent link="base_link"/>
         <child link="rear_hokuyo_link"/>
-        <origin xyz="-0.27 0 0.175" rpy="0 0 ${pi}"/>
+        <origin xyz="-0.27 0 0.165" rpy="0 0 ${pi}"/>
     </joint>
     <link name="omni_wheel_1">
