Commit message: update params

File: living_lab_robot_description/urdf/head_assy.urdf.xacro (robot description, xacro)
@@ -70,5 +70,5 @@
         <inertial>
             <origin xyz="0 0 0" rpy="0 0 0"/>
-            <mass value="1.0"/>
+            <mass value="5.0"/>
             <inertia ixx="1.0" ixy="0.0" ixz="0.0" iyy="1.0" iyz="0.0" izz="1.0"/>
         </inertial>
@@ -79,5 +79,5 @@
         <origin xyz="0.098 0 -0.016" rpy="0 0 0"/>
         <axis xyz="0 1 0"/>
-        <limit lower="${0/180*pi}" upper="${25/180*pi}" velocity="2.0" effort="1000"/>
+        <limit lower="${0/180*pi}" upper="${25/180*pi}" velocity="0.2" effort="1000"/>
     </joint>
     <xacro:insert_position_transmission name="head_tilt_unit_joint" />

Commit message: Change joint name

File: living_lab_robot_description/urdf/head_assy.urdf.xacro (robot description, xacro)
@@ -74,5 +74,5 @@
         </inertial>
     </link>
-    <joint name="head_tilt_unit_joint" type="revolute">
+    <joint name="head_tilt_joint" type="revolute">
         <parent link="head_assy"/>
         <child link="head_tilt_unit"/>
@@ -81,5 +81,5 @@
         <limit lower="${0/180*pi}" upper="${25/180*pi}" velocity="0.2" effort="1000"/>
     </joint>
-    <xacro:insert_position_transmission name="head_tilt_unit_joint" />
+    <xacro:insert_position_transmission name="head_tilt_joint" />
     <link name="head_d435_link">
         <visual>

Commit message: Add gaze_sync function & bug fixed
Use throttle tools for point cloud

File: living_lab_robot_description/urdf/head_assy.urdf.xacro (robot description, xacro)
@@ -95,7 +95,7 @@
     </link>
     <joint name="gaze_fixed_joint" type="fixed">
-        <parent link="head_tilt_unit"/>
+        <parent link="head_assy"/>
         <child link="gaze_link"/>
-        <origin xyz="0.04 0 0.0185" rpy="0 0 0"/>
+        <origin xyz="0.1 0 0.0185" rpy="0 0 0"/>
     </joint>
 </robot>
