Commit message: Add head_pan_controller for compensation of rotate body

File: living_lab_robot_description/urdf/body_assy.urdf.xacro (robot description, xacro)
@@ -25,5 +25,5 @@
         <origin xyz="0 0 0.272" rpy="0 0 0"/>
         <axis xyz="0 0 1"/>
-        <limit lower="${-200/180*pi}" upper="${200/180*pi}" velocity="1.0" effort="1000"/>
+        <limit lower="${-270/180*pi}" upper="${270/180*pi}" velocity="1.0" effort="1000"/>
     </joint>
     <xacro:insert_position_transmission name="body_rotate_joint" />

File: living_lab_robot_description/urdf/head1_assy.urdf.xacro (robot description, xacro)
@@ -25,5 +25,5 @@
         <origin xyz="0 0 0.660" rpy="0 0 0"/>
         <axis xyz="0 0 1"/>
-        <limit lower="${-90/180*pi}" upper="${90/180*pi}" velocity="1.0" effort="1000"/>
+        <limit lower="${-270/180*pi}" upper="${270/180*pi}" velocity="2.0" effort="1000"/>
     </joint>
     <xacro:insert_position_transmission name="head1_pan_joint" />

File: living_lab_robot_description/urdf/head2_assy.urdf.xacro (robot description, xacro)
@@ -25,5 +25,5 @@
         <origin xyz="0 0 0.9383" rpy="0 0 0"/>
         <axis xyz="0 0 1"/>
-        <limit lower="${-90/180*pi}" upper="${90/180*pi}" velocity="1.0" effort="1000"/>
+        <limit lower="${-270/180*pi}" upper="${270/180*pi}" velocity="2.0" effort="1000"/>
     </joint>
     <xacro:insert_position_transmission name="head2_pan_joint" />
@@ -48,4 +48,11 @@
     </link>
     <xacro:insert_rgbd_camera_sensor name="head2_d435"/>
+    <link name="gaze_link">
+        <inertial>
+            <origin xyz="0 0 0" rpy="0 0 0"/>
+            <mass value="1.0"/>
+            <inertia ixx="1.0" ixy="0.0" ixz="0.0" iyy="1.0" iyz="0.0" izz="1.0"/>
+        </inertial>
+    </link>
     <joint name="head2_d435_tilt_joint" type="revolute">
         <parent link="head2_assy"/>
@@ -53,6 +60,11 @@
         <origin xyz="0.126 0 0.07" rpy="0 0 0"/>
         <axis xyz="0 1 0"/>
-        <limit lower="${-10/180*pi}" upper="${40/180*pi}" velocity="1.0" effort="1000"/>
+        <limit lower="${-10/180*pi}" upper="${45/180*pi}" velocity="2.0" effort="1000"/>
     </joint>
     <xacro:insert_position_transmission name="head2_d435_tilt_joint" />
+    <joint name="gaze_fixed_joint" type="fixed">
+        <parent link="head2_assy"/>
+        <child link="gaze_link"/>
+        <origin xyz="0.126 0 0.07" rpy="0 0 0"/>
+    </joint>
 </robot>

Commit message: 설계 수정 사항 반영

File: living_lab_robot_description/urdf/body_assy.urdf.xacro (robot description, xacro)
@@ -5,5 +5,5 @@
             <origin xyz="0 0 0" rpy="0 0 0"/>
             <geometry>
-                <mesh filename="package://living_lab_robot_description/meshes/c3_body_assy.dae" scale="1 1 1"/>
+                <mesh filename="package://living_lab_robot_description/meshes/c4_body_assy.dae" scale="1 1 1"/>
             </geometry>
         </visual>
@@ -11,5 +11,5 @@
             <origin xyz="0 0 0" rpy="0 0 0"/>
             <geometry>
-                <mesh filename="package://living_lab_robot_description/meshes/c3_body_assy.dae" scale="1 1 1"/>
+                <mesh filename="package://living_lab_robot_description/meshes/c4_body_assy.dae" scale="1 1 1"/>
             </geometry>
         </collision>
@@ -23,14 +23,14 @@
         <parent link="base_link"/>
         <child link="body_assy"/>
-        <origin xyz="0 0 0.272" rpy="0 0 0"/>
+        <origin xyz="0 0 0.242" rpy="0 0 0"/>
         <axis xyz="0 0 1"/>
         <limit lower="${-270/180*pi}" upper="${270/180*pi}" velocity="1.0" effort="1000"/>
     </joint>
     <xacro:insert_position_transmission name="body_rotate_joint" />
-    <link name="elv_frame_assy">
+    <link name="trans_module">
         <visual>
             <origin xyz="0 0 0" rpy="0 0 0"/>
             <geometry>
-                <mesh filename="package://living_lab_robot_description/meshes/c3_elv_frame_assy.dae" scale="1 1 1"/>
+                <mesh filename="package://living_lab_robot_description/meshes/c4_trans_module.dae" scale="1 1 1"/>
             </geometry>
         </visual>
@@ -38,5 +38,5 @@
             <origin xyz="0 0 0" rpy="0 0 0"/>
             <geometry>
-                <mesh filename="package://living_lab_robot_description/meshes/c3_elv_frame_assy.dae" scale="1 1 1"/>
+                <mesh filename="package://living_lab_robot_description/meshes/c4_trans_module.dae" scale="1 1 1"/>
             </geometry>
         </collision>
@@ -47,11 +47,11 @@
         </inertial>
     </link>
-    <joint name="elv_frame_updown_joint" type="prismatic">
+    <joint name="trans_module_elv_joint" type="prismatic">
         <parent link="body_assy"/>
-        <child link="elv_frame_assy"/>
-        <origin xyz="0 0 0.400" rpy="0 0 0"/>
+        <child link="trans_module"/>
+        <origin xyz="-0.05 0 0.470" rpy="0 0 0"/>
         <axis xyz="0 0 1"/>
-        <limit lower="-0.25" upper="0.15" velocity="1.0" effort="1000"/>
+        <limit lower="-0.25" upper="0.1" velocity="1.0" effort="1000"/>
     </joint>
-    <xacro:insert_position_transmission name="elv_frame_updown_joint" />
+    <xacro:insert_position_transmission name="trans_module_elv_joint" />
 </robot>

File: living_lab_robot_description/urdf/mobile_assy.urdf.xacro (robot description, xacro)
@@ -13,5 +13,5 @@
             <origin xyz="0 0 0" rpy="0 0 0"/>
             <geometry>
-                <mesh filename="package://living_lab_robot_description/meshes/c3_mobile_assy.dae" scale="1 1 1"/>
+                <mesh filename="package://living_lab_robot_description/meshes/c4_mobile_assy.dae" scale="1 1 1"/>
             </geometry>
         </visual>
@@ -19,10 +19,10 @@
             <origin xyz="0 0 0" rpy="0 0 0"/>
             <geometry>
-                <mesh filename="package://living_lab_robot_description/meshes/c3_mobile_assy.dae" scale="1 1 1"/>
+                <mesh filename="package://living_lab_robot_description/meshes/c4_mobile_assy.dae" scale="1 1 1"/>
             </geometry>
         </collision>
         <inertial>
             <origin xyz="0 0 0" rpy="0 0 0"/>
-            <mass value="1.0"/>
+            <mass value="30.0"/>
             <inertia ixx="10.0" ixy="0.0" ixz="0.0" iyy="10.0" iyz="0.0" izz="10.0"/>
         </inertial>
@@ -59,3 +59,81 @@
         <origin xyz="-0.27 0 0.175" rpy="0 0 ${pi}"/>
     </joint>
+    <link name="omni_wheel_1">
+        <visual>
+            <origin xyz="0 0 0" rpy="0 0 0"/>
+            <geometry>
+                <mesh filename="package://living_lab_robot_description/meshes/omni_wheel.dae" scale="1 1 1"/>
+            </geometry>
+        </visual>
+        <collision>
+            <origin xyz="0 0 0" rpy="0 0 0"/>
+            <geometry>
+                <mesh filename="package://living_lab_robot_description/meshes/omni_wheel.dae" scale="1 1 1"/>
+            </geometry>
+        </collision>
+        <inertial>
+            <origin xyz="0 0 0" rpy="0 0 0"/>
+            <mass value="1.0"/>
+            <inertia ixx="1.0" ixy="0.0" ixz="0.0" iyy="1.0" iyz="0.0" izz="1.0"/>
+        </inertial>
+    </link>
+    <joint name="omni_wheel_1_joint" type="continuous">
+        <parent link="base_link"/>
+        <child link="omni_wheel_1"/>
+        <origin xyz="${0.282 * cos(pi/3)}  ${0.282 * sin(pi/3)} 0" rpy="0 0 ${-pi/6}"/>
+        <axis xyz="0 1 0"/>
+    </joint>
+    <xacro:insert_velocity_transmission name="omni_wheel_1_joint" />
+    <link name="omni_wheel_2">
+        <visual>
+            <origin xyz="0 0 0" rpy="0 0 0"/>
+            <geometry>
+                <mesh filename="package://living_lab_robot_description/meshes/omni_wheel.dae" scale="1 1 1"/>
+            </geometry>
+        </visual>
+        <collision>
+            <origin xyz="0 0 0" rpy="0 0 0"/>
+            <geometry>
+                <mesh filename="package://living_lab_robot_description/meshes/omni_wheel.dae" scale="1 1 1"/>
+            </geometry>
+        </collision>
+        <inertial>
+            <origin xyz="0 0 0" rpy="0 0 0"/>
+            <mass value="1.0"/>
+            <inertia ixx="1.0" ixy="0.0" ixz="0.0" iyy="1.0" iyz="0.0" izz="1.0"/>
+        </inertial>
+    </link>
+    <joint name="omni_wheel_2_joint" type="continuous">
+        <parent link="base_link"/>
+        <child link="omni_wheel_2"/>
+        <origin xyz="${0.282 * cos(pi/3)}  ${0.282 * sin(-pi/3)} 0" rpy="0 0 ${-5*pi/6}"/>
+        <axis xyz="0 1 0"/>
+    </joint>
+    <xacro:insert_velocity_transmission name="omni_wheel_2_joint" />
+    <link name="omni_wheel_3">
+        <visual>
+            <origin xyz="0 0 0" rpy="0 0 0"/>
+            <geometry>
+                <mesh filename="package://living_lab_robot_description/meshes/omni_wheel.dae" scale="1 1 1"/>
+            </geometry>
+        </visual>
+        <collision>
+            <origin xyz="0 0 0" rpy="0 0 0"/>
+            <geometry>
+                <mesh filename="package://living_lab_robot_description/meshes/omni_wheel.dae" scale="1 1 1"/>
+            </geometry>
+        </collision>
+        <inertial>
+            <origin xyz="0 0 0" rpy="0 0 0"/>
+            <mass value="1.0"/>
+            <inertia ixx="1.0" ixy="0.0" ixz="0.0" iyy="1.0" iyz="0.0" izz="1.0"/>
+        </inertial>
+    </link>
+    <joint name="omni_wheel_3_joint" type="continuous">
+        <parent link="base_link"/>
+        <child link="omni_wheel_3"/>
+        <origin xyz="-0.282 0 0" rpy="0 0 ${pi/2}"/>
+        <axis xyz="0 1 0"/>
+    </joint>
+    <xacro:insert_velocity_transmission name="omni_wheel_3_joint" />
 </robot>

File: living_lab_robot_description/urdf/robot.urdf.xacro (robot description, xacro)
@@ -5,7 +5,6 @@
     <xacro:include filename="$(find living_lab_robot_description)/urdf/mobile_assy.urdf.xacro"/>
     <xacro:include filename="$(find living_lab_robot_description)/urdf/body_assy.urdf.xacro"/>
-    <xacro:include filename="$(find living_lab_robot_description)/urdf/robotis_arm.urdf.xacro"/>
-    <xacro:include filename="$(find living_lab_robot_description)/urdf/robotis_gripper.urdf.xacro"/>
-    <xacro:include filename="$(find living_lab_robot_description)/urdf/head1_assy.urdf.xacro"/>
-    <xacro:include filename="$(find living_lab_robot_description)/urdf/head2_assy.urdf.xacro"/>
+    <xacro:include filename="$(find living_lab_robot_description)/urdf/manipulator_arm.urdf.xacro"/>
+    <xacro:include filename="$(find living_lab_robot_description)/urdf/gripper.urdf.xacro"/>
+    <xacro:include filename="$(find living_lab_robot_description)/urdf/head_assy.urdf.xacro"/>
 </robot>

Commit message: Change the joint name

File: living_lab_robot_description/urdf/body_assy.urdf.xacro (robot description, xacro)
@@ -47,5 +47,5 @@
         </inertial>
     </link>
-    <joint name="trans_module_elv_joint" type="prismatic">
+    <joint name="elavation_joint" type="prismatic">
         <parent link="body_assy"/>
         <child link="trans_module"/>
@@ -54,4 +54,4 @@
         <limit lower="-0.25" upper="0.1" velocity="1.0" effort="1000"/>
     </joint>
-    <xacro:insert_position_transmission name="trans_module_elv_joint" />
+    <xacro:insert_position_transmission name="elavation_joint" />
 </robot>

File: living_lab_robot_description/urdf/manipulator_arm.urdf.xacro (robot description, xacro)
@@ -47,5 +47,5 @@
         </inertial>
     </link>
-    <joint name="arm_joint1" type="revolute">
+    <joint name="arm1_joint" type="revolute">
         <parent link="manipulator_base"/>
         <child link="manipulator_link1"/>
@@ -54,8 +54,8 @@
         <limit lower="${-90/180*pi}" upper="${90/180*pi}" velocity="1.0" effort="1000"/>
     </joint>
-    <xacro:insert_position_transmission name="arm_joint1" />
+    <xacro:insert_position_transmission name="arm1_joint" />
     <link name="manipulator_link2">
         <visual>
-            <origin xyz="0 0 0" rpy="0 0 0"/>
+            <origin xyz="0 0 0" rpy="0 ${-90/180*pi} 0"/>
             <geometry>
                 <mesh filename="package://living_lab_robot_description/meshes/manipulator_link2.dae" scale="1 1 1"/>
@@ -63,5 +63,5 @@
         </visual>
         <collision>
-            <origin xyz="0 0 0" rpy="0 0 0"/>
+            <origin xyz="0 0 0" rpy="0 ${-90/180*pi} 0"/>
             <geometry>
                 <mesh filename="package://living_lab_robot_description/meshes/manipulator_link2.dae" scale="1 1 1"/>
@@ -74,5 +74,5 @@
         </inertial>
     </link>
-    <joint name="arm_joint2" type="revolute">
+    <joint name="arm2_joint" type="revolute">
         <parent link="manipulator_link1"/>
         <child link="manipulator_link2"/>
@@ -81,8 +81,8 @@
         <limit lower="${-190/180*pi}" upper="${10/180*pi}" velocity="1.0" effort="1000"/>
     </joint>
-    <xacro:insert_position_transmission name="arm_joint2" />
+    <xacro:insert_position_transmission name="arm2_joint" />
     <link name="manipulator_link3">
         <visual>
-            <origin xyz="0 0 0" rpy="0 0 0"/>
+            <origin xyz="0 0 0" rpy="0 ${90/180*pi} 0"/>
             <geometry>
                 <mesh filename="package://living_lab_robot_description/meshes/manipulator_link3.dae" scale="1 1 1"/>
@@ -90,5 +90,5 @@
         </visual>
         <collision>
-            <origin xyz="0 0 0" rpy="0 0 0"/>
+            <origin xyz="0 0 0" rpy="0 ${90/180*pi} 0"/>
             <geometry>
                 <mesh filename="package://living_lab_robot_description/meshes/manipulator_link3.dae" scale="1 1 1"/>
@@ -101,12 +101,12 @@
         </inertial>
     </link>
-    <joint name="arm_joint3" type="revolute">
+    <joint name="arm3_joint" type="revolute">
         <parent link="manipulator_link2"/>
         <child link="manipulator_link3"/>
-        <origin xyz="0.030 0 -0.264" rpy="0 0 0"/>
+        <origin xyz="0.264 0 0.030" rpy="0 0 0"/>
         <axis xyz="0 1 0"/>
         <limit lower="${0/180*pi}" upper="${240/180*pi}" velocity="1.0" effort="1000"/>
     </joint>
-    <xacro:insert_position_transmission name="arm_joint3" />
+    <xacro:insert_position_transmission name="arm3_joint" />
     <link name="manipulator_link4">
         <visual>
@@ -128,12 +128,12 @@
         </inertial>
     </link>
-    <joint name="arm_joint4" type="revolute">
+    <joint name="arm4_joint" type="revolute">
         <parent link="manipulator_link3"/>
         <child link="manipulator_link4"/>
-        <origin xyz="0.042 0 0.231" rpy="0 0 0"/>
+        <origin xyz="0.231 0 0.042" rpy="0 0 0"/>
         <axis xyz="0 0 1"/>
         <limit lower="${-180/180*pi}" upper="${180/180*pi}" velocity="1.0" effort="1000"/>
     </joint>
-    <xacro:insert_position_transmission name="arm_joint4" />
+    <xacro:insert_position_transmission name="arm4_joint" />
     <link name="manipulator_link5">
         <visual>
@@ -155,5 +155,5 @@
         </inertial>
     </link>
-    <joint name="arm_joint5" type="revolute">
+    <joint name="arm5_joint" type="revolute">
         <parent link="manipulator_link4"/>
         <child link="manipulator_link5"/>
@@ -162,5 +162,5 @@
         <limit lower="${-180/180*pi}" upper="${180/180*pi}" velocity="1.0" effort="1000"/>
     </joint>
-    <xacro:insert_position_transmission name="arm_joint5" />
+    <xacro:insert_position_transmission name="arm5_joint" />
     <link name="manipulator_link6">
         <inertial>
@@ -170,5 +170,5 @@
         </inertial>
     </link>
-    <joint name="arm_joint6" type="revolute">
+    <joint name="arm6_joint" type="revolute">
         <parent link="manipulator_link5"/>
         <child link="manipulator_link6"/>
@@ -177,4 +177,4 @@
         <limit lower="${-180/180*pi}" upper="${180/180*pi}" velocity="1.0" effort="1000"/>
     </joint>
-    <xacro:insert_position_transmission name="arm_joint6" />
+    <xacro:insert_position_transmission name="arm6_joint" />
 </robot>

Commit message: Change the joint name

File: living_lab_robot_description/urdf/body_assy.urdf.xacro (robot description, xacro)
@@ -47,5 +47,5 @@
         </inertial>
     </link>
-    <joint name="elavation_joint" type="prismatic">
+    <joint name="elevation_joint" type="prismatic">
         <parent link="body_assy"/>
         <child link="trans_module"/>
@@ -54,4 +54,4 @@
         <limit lower="-0.25" upper="0.1" velocity="1.0" effort="1000"/>
     </joint>
-    <xacro:insert_position_transmission name="elavation_joint" />
+    <xacro:insert_position_transmission name="elevation_joint" />
 </robot>

Commit message: add dynamixel bringup package

File: living_lab_robot_description/urdf/body_assy.urdf.xacro (robot description, xacro)
@@ -50,7 +50,7 @@
         <parent link="body_assy"/>
         <child link="trans_module"/>
-        <origin xyz="-0.05 0 0.470" rpy="0 0 0"/>
+        <origin xyz="-0.05 0 0.650" rpy="0 0 0"/>
         <axis xyz="0 0 1"/>
-        <limit lower="-0.25" upper="0.1" velocity="1.0" effort="1000"/>
+        <limit lower="-0.40" upper="0" velocity="1.0" effort="1000"/>
     </joint>
     <xacro:insert_position_transmission name="elevation_joint" />

File: living_lab_robot_description/urdf/gripper.urdf.xacro (robot description, xacro)
@@ -3,5 +3,5 @@
     <link name="gripper">
         <visual>
-            <origin xyz="0 0 0" rpy="0 0 0"/>
+            <origin xyz="0 0 0" rpy="0 ${90/180*pi} 0"/>
             <geometry>
                 <mesh filename="package://living_lab_robot_description/meshes/gripper.dae" scale="1 1 1"/>
@@ -9,5 +9,5 @@
         </visual>
         <collision>
-            <origin xyz="0 0 0" rpy="0 0 0"/>
+            <origin xyz="0 0 0" rpy="0 ${90/180*pi} 0"/>
             <geometry>
                 <mesh filename="package://living_lab_robot_description/meshes/gripper.dae" scale="1 1 1"/>
@@ -35,5 +35,5 @@
         <parent link="gripper"/>
         <child link="end_effector"/>
-        <origin xyz="0 0 0.096" rpy="0 0 0"/>
+        <origin xyz="0.096 0 0" rpy="0 0 0"/>
     </joint>
 </robot>

File: living_lab_robot_description/urdf/manipulator_arm.urdf.xacro (robot description, xacro)
@@ -23,7 +23,7 @@
         <parent link="trans_module"/>
         <child link="manipulator_base"/>
-        <origin xyz="-0.116 0 -0.0228" rpy="0 0 0"/>
+        <origin xyz="0.04 0 -0.0228" rpy="0 0 0"/>
         <axis xyz="1 0 0"/>
-        <limit lower="0" upper="0.15" velocity="1.0" effort="1000"/>
+        <limit lower="-0.14" upper="0" velocity="1.0" effort="1000"/>
     </joint>
     <xacro:insert_position_transmission name="arm_base_joint" />
@@ -79,5 +79,5 @@
         <origin xyz="0.033 0 0" rpy="0 0 0"/>
         <axis xyz="0 1 0"/>
-        <limit lower="${-190/180*pi}" upper="${10/180*pi}" velocity="1.0" effort="1000"/>
+        <limit lower="${-90/180*pi}" upper="${90/180*pi}" velocity="1.0" effort="1000"/>
     </joint>
     <xacro:insert_position_transmission name="arm2_joint" />
@@ -106,10 +106,10 @@
         <origin xyz="0.264 0 0.030" rpy="0 0 0"/>
         <axis xyz="0 1 0"/>
-        <limit lower="${0/180*pi}" upper="${240/180*pi}" velocity="1.0" effort="1000"/>
+        <limit lower="${-180/180*pi}" upper="${5/180*pi}" velocity="1.0" effort="1000"/>
     </joint>
     <xacro:insert_position_transmission name="arm3_joint" />
     <link name="manipulator_link4">
         <visual>
-            <origin xyz="0 0 0" rpy="0 0 0"/>
+            <origin xyz="0 0 0" rpy="0 ${90/180*pi} 0"/>
             <geometry>
                 <mesh filename="package://living_lab_robot_description/meshes/manipulator_link4.dae" scale="1 1 1"/>
@@ -117,5 +117,5 @@
         </visual>
         <collision>
-            <origin xyz="0 0 0" rpy="0 0 0"/>
+            <origin xyz="0 0 0" rpy="0 ${90/180*pi} 0"/>
             <geometry>
                 <mesh filename="package://living_lab_robot_description/meshes/manipulator_link4.dae" scale="1 1 1"/>
@@ -131,6 +131,6 @@
         <parent link="manipulator_link3"/>
         <child link="manipulator_link4"/>
-        <origin xyz="0.231 0 0.042" rpy="0 0 0"/>
-        <axis xyz="0 0 1"/>
+        <origin xyz="0.231 0 -0.042" rpy="0 0 0"/>
+        <axis xyz="1 0 0"/>
         <limit lower="${-180/180*pi}" upper="${180/180*pi}" velocity="1.0" effort="1000"/>
     </joint>
@@ -138,5 +138,5 @@
     <link name="manipulator_link5">
         <visual>
-            <origin xyz="0 0 0" rpy="0 0 0"/>
+            <origin xyz="0 0 0" rpy="0 ${90/180*pi} 0"/>
             <geometry>
                 <mesh filename="package://living_lab_robot_description/meshes/manipulator_link5.dae" scale="1 1 1"/>
@@ -144,5 +144,5 @@
         </visual>
         <collision>
-            <origin xyz="0 0 0" rpy="0 0 0"/>
+            <origin xyz="0 0 0" rpy="0 ${90/180*pi} 0"/>
             <geometry>
                 <mesh filename="package://living_lab_robot_description/meshes/manipulator_link5.dae" scale="1 1 1"/>
@@ -158,7 +158,7 @@
         <parent link="manipulator_link4"/>
         <child link="manipulator_link5"/>
-        <origin xyz="0 0 0.027" rpy="0 0 0"/>
+        <origin xyz="0.027 0 0" rpy="0 0 0"/>
         <axis xyz="0 1 0"/>
-        <limit lower="${-180/180*pi}" upper="${180/180*pi}" velocity="1.0" effort="1000"/>
+        <limit lower="${-90/180*pi}" upper="${90/180*pi}" velocity="1.0" effort="1000"/>
     </joint>
     <xacro:insert_position_transmission name="arm5_joint" />
@@ -173,6 +173,6 @@
         <parent link="manipulator_link5"/>
         <child link="manipulator_link6"/>
-        <origin xyz="0 0 0.123" rpy="0 0 0"/>
-        <axis xyz="0 0 1"/>
+        <origin xyz="0.123 0 0" rpy="0 0 0"/>
+        <axis xyz="1 0 0"/>
         <limit lower="${-180/180*pi}" upper="${180/180*pi}" velocity="1.0" effort="1000"/>
     </joint>

Commit message: change the limit of joints

File: living_lab_robot_description/urdf/body_assy.urdf.xacro (robot description, xacro)
@@ -52,5 +52,5 @@
         <origin xyz="-0.05 0 0.650" rpy="0 0 0"/>
         <axis xyz="0 0 1"/>
-        <limit lower="-0.40" upper="0" velocity="1.0" effort="1000"/>
+        <limit lower="-0.45" upper="0" velocity="1.0" effort="1000"/>
     </joint>
     <xacro:insert_position_transmission name="elevation_joint" />

File: living_lab_robot_description/urdf/manipulator_arm.urdf.xacro (robot description, xacro)
@@ -25,5 +25,5 @@
         <origin xyz="0.04 0 -0.0228" rpy="0 0 0"/>
         <axis xyz="1 0 0"/>
-        <limit lower="-0.14" upper="0" velocity="1.0" effort="1000"/>
+        <limit lower="-0.15" upper="0" velocity="1.0" effort="1000"/>
     </joint>
     <xacro:insert_position_transmission name="arm_base_joint" />
