Commit message: Change the range of joints

File: living_lab_robot_description/urdf/body_assy.urdf.xacro (robot description, xacro)
@@ -25,5 +25,5 @@
         <origin xyz="0 0 0.242" rpy="0 0 0"/>
         <axis xyz="0 0 1"/>
-        <limit lower="${-270/180*pi}" upper="${270/180*pi}" velocity="1.0" effort="1000"/>
+        <limit lower="${-180/180*pi}" upper="${180/180*pi}" velocity="1.0" effort="1000"/>
     </joint>
     <xacro:insert_position_transmission name="body_rotate_joint" />
@@ -52,5 +52,5 @@
         <origin xyz="-0.05 0 0.650" rpy="0 0 0"/>
         <axis xyz="0 0 1"/>
-        <limit lower="-0.45" upper="0" velocity="1.0" effort="1000"/>
+        <limit lower="-0.45" upper="0" velocity="0.02" effort="1000"/>
     </joint>
     <xacro:insert_position_transmission name="elevation_joint" />

File: living_lab_robot_description/urdf/gripper.urdf.xacro (robot description, xacro)
@@ -32,5 +32,5 @@
         </inertial>
     </link>
-    <joint name="end_effector_joint" type="fixed">
+    <joint name="gripper_joint" type="fixed">
         <parent link="gripper"/>
         <child link="end_effector"/>

File: living_lab_robot_description/urdf/manipulator_arm.urdf.xacro (robot description, xacro)
@@ -52,5 +52,5 @@
         <origin xyz="0.15612 0 -0.051215" rpy="0 0 0"/>
         <axis xyz="1 0 0"/>
-        <limit lower="${-90/180*pi}" upper="${90/180*pi}" velocity="1.0" effort="1000"/>
+        <limit lower="${-90/180*pi}" upper="${90/180*pi}" velocity="0.4" effort="1000"/>
     </joint>
     <xacro:insert_position_transmission name="arm1_joint" />
@@ -79,5 +79,5 @@
         <origin xyz="0.033 0 0" rpy="0 0 0"/>
         <axis xyz="0 1 0"/>
-        <limit lower="${-90/180*pi}" upper="${90/180*pi}" velocity="1.0" effort="1000"/>
+        <limit lower="${-96/180*pi}" upper="${96/180*pi}" velocity="0.4" effort="1000"/>
     </joint>
     <xacro:insert_position_transmission name="arm2_joint" />
@@ -106,5 +106,5 @@
         <origin xyz="0.264 0 0.030" rpy="0 0 0"/>
         <axis xyz="0 1 0"/>
-        <limit lower="${-180/180*pi}" upper="${5/180*pi}" velocity="1.0" effort="1000"/>
+        <limit lower="${-180/180*pi}" upper="${5/180*pi}" velocity="0.4" effort="1000"/>
     </joint>
     <xacro:insert_position_transmission name="arm3_joint" />
@@ -133,5 +133,5 @@
         <origin xyz="0.231 0 -0.042" rpy="0 0 0"/>
         <axis xyz="1 0 0"/>
-        <limit lower="${-180/180*pi}" upper="${180/180*pi}" velocity="1.0" effort="1000"/>
+        <limit lower="${-180/180*pi}" upper="${180/180*pi}" velocity="0.4" effort="1000"/>
     </joint>
     <xacro:insert_position_transmission name="arm4_joint" />
@@ -160,5 +160,5 @@
         <origin xyz="0.027 0 0" rpy="0 0 0"/>
         <axis xyz="0 1 0"/>
-        <limit lower="${-90/180*pi}" upper="${90/180*pi}" velocity="1.0" effort="1000"/>
+        <limit lower="${-90/180*pi}" upper="${90/180*pi}" velocity="0.4" effort="1000"/>
     </joint>
     <xacro:insert_position_transmission name="arm5_joint" />
@@ -175,5 +175,5 @@
         <origin xyz="0.123 0 0" rpy="0 0 0"/>
         <axis xyz="1 0 0"/>
-        <limit lower="${-180/180*pi}" upper="${180/180*pi}" velocity="1.0" effort="1000"/>
+        <limit lower="${-180/180*pi}" upper="${180/180*pi}" velocity="0.4" effort="1000"/>
     </joint>
     <xacro:insert_position_transmission name="arm6_joint" />

File: living_lab_robot_description/urdf/mobile_assy.urdf.xacro (robot description, xacro)
@@ -31,5 +31,5 @@
         <parent link="base_footprint"/>
         <child link="base_link"/>
-        <origin xyz="0 0 0.0635" rpy="0 0 0"/>
+        <origin xyz="0 0 0.0645" rpy="0 0 0"/>
     </joint>
     <link name="front_hokuyo_link">

Commit message: adjust parameters

File: living_lab_robot_description/urdf/body_assy.urdf.xacro (robot description, xacro)
@@ -52,5 +52,5 @@
         <origin xyz="-0.05 0 0.650" rpy="0 0 0"/>
         <axis xyz="0 0 1"/>
-        <limit lower="-0.45" upper="0" velocity="0.02" effort="1000"/>
+        <limit lower="-0.45" upper="0" velocity="0.04" effort="1000"/>
     </joint>
     <xacro:insert_position_transmission name="elevation_joint" />

File: living_lab_robot_description/urdf/manipulator_arm.urdf.xacro (robot description, xacro)
@@ -52,5 +52,5 @@
         <origin xyz="0.15612 0 -0.051215" rpy="0 0 0"/>
         <axis xyz="1 0 0"/>
-        <limit lower="${-90/180*pi}" upper="${90/180*pi}" velocity="0.4" effort="1000"/>
+        <limit lower="${-180/180*pi}" upper="${180/180*pi}" velocity="0.4" effort="1000"/>
     </joint>
     <xacro:insert_position_transmission name="arm1_joint" />
@@ -160,5 +160,5 @@
         <origin xyz="0.027 0 0" rpy="0 0 0"/>
         <axis xyz="0 1 0"/>
-        <limit lower="${-90/180*pi}" upper="${90/180*pi}" velocity="0.4" effort="1000"/>
+        <limit lower="${-95/180*pi}" upper="${95/180*pi}" velocity="0.4" effort="1000"/>
     </joint>
     <xacro:insert_position_transmission name="arm5_joint" />

Commit message: Add rosbridge & adjust value of joint location

File: living_lab_robot_description/urdf/body_assy.urdf.xacro (robot description, xacro)
@@ -50,5 +50,5 @@
         <parent link="body_assy"/>
         <child link="trans_module"/>
-        <origin xyz="-0.05 0 0.650" rpy="0 0 0"/>
+        <origin xyz="-0.05 0 0.660" rpy="0 0 0"/>
         <axis xyz="0 0 1"/>
         <limit lower="-0.45" upper="0" velocity="0.04" effort="1000"/>

Commit message: update collada model and urdf

File: living_lab_robot_description/urdf/body_assy.urdf.xacro (robot description, xacro)
@@ -5,5 +5,5 @@
             <origin xyz="0 0 0" rpy="0 0 0"/>
             <geometry>
-                <mesh filename="package://living_lab_robot_description/meshes/c4_body_assy.dae" scale="1 1 1"/>
+                <mesh filename="package://living_lab_robot_description/meshes/body_assy.dae" scale="1 1 1"/>
             </geometry>
         </visual>
@@ -11,5 +11,5 @@
             <origin xyz="0 0 0" rpy="0 0 0"/>
             <geometry>
-                <mesh filename="package://living_lab_robot_description/meshes/c4_body_assy.dae" scale="1 1 1"/>
+                <mesh filename="package://living_lab_robot_description/meshes/body_assy.dae" scale="1 1 1"/>
             </geometry>
         </collision>
@@ -25,12 +25,12 @@
         <origin xyz="0 0 0.242" rpy="0 0 0"/>
         <axis xyz="0 0 1"/>
-        <limit lower="${-180/180*pi}" upper="${180/180*pi}" velocity="1.0" effort="1000"/>
+        <limit lower="${-200/180*pi}" upper="${200/180*pi}" velocity="1.0" effort="1000"/>
     </joint>
     <xacro:insert_position_transmission name="body_rotate_joint" />
-    <link name="trans_module">
+    <link name="elevation_module">
         <visual>
             <origin xyz="0 0 0" rpy="0 0 0"/>
             <geometry>
-                <mesh filename="package://living_lab_robot_description/meshes/c4_trans_module.dae" scale="1 1 1"/>
+                <mesh filename="package://living_lab_robot_description/meshes/elevation_module.dae" scale="1 1 1"/>
             </geometry>
         </visual>
@@ -38,5 +38,5 @@
             <origin xyz="0 0 0" rpy="0 0 0"/>
             <geometry>
-                <mesh filename="package://living_lab_robot_description/meshes/c4_trans_module.dae" scale="1 1 1"/>
+                <mesh filename="package://living_lab_robot_description/meshes/elevation_module.dae" scale="1 1 1"/>
             </geometry>
         </collision>
@@ -49,6 +49,6 @@
     <joint name="elevation_joint" type="prismatic">
         <parent link="body_assy"/>
-        <child link="trans_module"/>
-        <origin xyz="-0.05 0 0.660" rpy="0 0 0"/>
+        <child link="elevation_module"/>
+        <origin xyz="-0.05 0 0.665" rpy="0 0 0"/>
         <axis xyz="0 0 1"/>
         <limit lower="-0.45" upper="0" velocity="0.04" effort="1000"/>

File: living_lab_robot_description/urdf/gripper.urdf.xacro (robot description, xacro)
@@ -3,5 +3,5 @@
     <link name="gripper">
         <visual>
-            <origin xyz="0 0 0" rpy="0 ${90/180*pi} 0"/>
+            <origin xyz="0 0 0" rpy="0 0 0"/>
             <geometry>
                 <mesh filename="package://living_lab_robot_description/meshes/gripper.dae" scale="1 1 1"/>
@@ -9,5 +9,5 @@
         </visual>
         <collision>
-            <origin xyz="0 0 0" rpy="0 ${90/180*pi} 0"/>
+            <origin xyz="0 0 0" rpy="0 0 0"/>
             <geometry>
                 <mesh filename="package://living_lab_robot_description/meshes/gripper.dae" scale="1 1 1"/>
@@ -21,5 +21,5 @@
     </link>
     <joint name="gripper_mount_joint" type="fixed">
-        <parent link="manipulator_link6"/>
+        <parent link="arm_link6"/>
         <child link="gripper"/>
         <origin xyz="0 0 0" rpy="0 0 0"/>

File: living_lab_robot_description/urdf/head_assy.urdf.xacro (robot description, xacro)
@@ -1,9 +1,10 @@
 <?xml version="1.0"?>
 <robot xmlns:xacro="http://www.ros.org/wiki/xacro">
+    <xacro:include filename="$(find realsense2_description)/urdf/_d435.urdf.xacro" />
     <link name="head_assy">
         <visual>
             <origin xyz="0 0 0" rpy="0 0 0"/>
             <geometry>
-                <mesh filename="package://living_lab_robot_description/meshes/c4_head_assy.dae" scale="1 1 1"/>
+                <mesh filename="package://living_lab_robot_description/meshes/head_assy.dae" scale="1 1 1"/>
             </geometry>
         </visual>
@@ -11,5 +12,5 @@
             <origin xyz="0 0 0" rpy="0 0 0"/>
             <geometry>
-                <mesh filename="package://living_lab_robot_description/meshes/c4_head_assy.dae" scale="1 1 1"/>
+                <mesh filename="package://living_lab_robot_description/meshes/head_assy.dae" scale="1 1 1"/>
             </geometry>
         </collision>
@@ -23,5 +24,5 @@
         <parent link="body_assy"/>
         <child link="head_assy"/>
-        <origin xyz="0 0 0.982" rpy="0 0 0"/>
+        <origin xyz="0 0 0.983" rpy="0 0 0"/>
         <axis xyz="0 0 1"/>
         <limit lower="${-270/180*pi}" upper="${270/180*pi}" velocity="2.0" effort="1000"/>
@@ -79,32 +80,11 @@
         <origin xyz="0.098 0 -0.016" rpy="0 0 0"/>
         <axis xyz="0 1 0"/>
-        <limit lower="${0/180*pi}" upper="${25/180*pi}" velocity="0.2" effort="1000"/>
+        <limit lower="${0/180*pi}" upper="${40/180*pi}" velocity="0.2" effort="1000"/>
     </joint>
     <xacro:insert_position_transmission name="head_tilt_joint" />
-    <link name="head_d435_link">
-        <visual>
-            <origin xyz="0 0 0" rpy="0 0 0"/>
-            <geometry>
-                <box size="0.025 0.090 0.025"/>
-            </geometry>
-        </visual>
-        <collision>
-            <origin xyz="0 0 0" rpy="0 0 0"/>
-            <geometry>
-                <box size="0.025 0.090 0.025"/>
-            </geometry>
-        </collision>
-        <inertial>
-            <origin xyz="0 0 0" rpy="0 0 0"/>
-            <mass value="1.0"/>
-            <inertia ixx="1.0" ixy="0.0" ixz="0.0" iyy="1.0" iyz="0.0" izz="1.0"/>
-        </inertial>
-    </link>
-    <xacro:insert_rgbd_camera_sensor name="head_d435"/>
-    <joint name="head_d435_mount_joint" type="fixed">
-        <parent link="head_tilt_unit"/>
-        <child link="head_d435_link"/>
-        <origin xyz="0.02 0 0.03085" rpy="0 0 0"/>
-    </joint>
+    <xacro:sensor_d435 parent="head_tilt_unit">
+        <origin xyz="0.0172 0 0.0185" rpy="0 0 0"/>
+    </xacro:sensor_d435>
+    <xacro:insert_rgbd_camera_sensor name="camera"/>
     <link name="gaze_link">
         <inertial>
@@ -117,5 +97,5 @@
         <parent link="head_tilt_unit"/>
         <child link="gaze_link"/>
-        <origin xyz="0.032 0 0.03085" rpy="0 0 0"/>
+        <origin xyz="0.04 0 0.0185" rpy="0 0 0"/>
     </joint>
 </robot>

File: living_lab_robot_description/urdf/mobile_assy.urdf.xacro (robot description, xacro)
@@ -1,17 +1,10 @@
 <?xml version="1.0"?>
 <robot xmlns:xacro="http://www.ros.org/wiki/xacro">
-    <link name="base_footprint">
-        <visual>
-            <origin xyz="0 0 0" rpy="0 0 0" />
-            <geometry>
-                <box size="0.001 0.001 0.001" />
-            </geometry>
-        </visual>
-    </link>
+    <link name="base_footprint"/>
     <link name="base_link">
         <visual>
             <origin xyz="0 0 0" rpy="0 0 0"/>
             <geometry>
-                <mesh filename="package://living_lab_robot_description/meshes/c4_mobile_assy.dae" scale="1 1 1"/>
+                <mesh filename="package://living_lab_robot_description/meshes/mobile_assy.dae" scale="1 1 1"/>
             </geometry>
         </visual>
@@ -19,5 +12,5 @@
             <origin xyz="0 0 0" rpy="0 0 0"/>
             <geometry>
-                <mesh filename="package://living_lab_robot_description/meshes/c4_mobile_assy.dae" scale="1 1 1"/>
+                <mesh filename="package://living_lab_robot_description/meshes/mobile_assy.dae" scale="1 1 1"/>
             </geometry>
         </collision>
@@ -31,5 +24,5 @@
         <parent link="base_footprint"/>
         <child link="base_link"/>
-        <origin xyz="0 0 0.0645" rpy="0 0 0"/>
+        <origin xyz="0 0 0.0635" rpy="0 0 0"/>
     </joint>
     <link name="front_hokuyo_link">

File: living_lab_robot_description/urdf/robot.urdf.xacro (robot description, xacro)
@@ -5,5 +5,5 @@
     <xacro:include filename="$(find living_lab_robot_description)/urdf/mobile_assy.urdf.xacro"/>
     <xacro:include filename="$(find living_lab_robot_description)/urdf/body_assy.urdf.xacro"/>
-    <xacro:include filename="$(find living_lab_robot_description)/urdf/manipulator_arm.urdf.xacro"/>
+    <xacro:include filename="$(find living_lab_robot_description)/urdf/arm.urdf.xacro"/>
     <xacro:include filename="$(find living_lab_robot_description)/urdf/gripper.urdf.xacro"/>
     <xacro:include filename="$(find living_lab_robot_description)/urdf/head_assy.urdf.xacro"/>

Commit message: Apply mass and inertia values for parts

File: living_lab_robot_description/urdf/body_assy.urdf.xacro (robot description, xacro)
@@ -15,7 +15,7 @@
         </collision>
         <inertial>
-            <origin xyz="0 0 0" rpy="0 0 0"/>
+            <origin xyz="0 0 0.3780" rpy="0 0 0"/>
             <mass value="5.0"/>
-            <inertia ixx="1.0" ixy="0.0" ixz="0.0" iyy="1.0" iyz="0.0" izz="1.0"/>
+            <inertia ixx="0.278381" ixy="0.0" ixz="0.0" iyy="0.278381" iyz="0.0" izz="0.080481"/>
         </inertial>
     </link>
@@ -43,6 +43,6 @@
         <inertial>
             <origin xyz="0 0 0" rpy="0 0 0"/>
-            <mass value="1.0"/>
-            <inertia ixx="1.0" ixy="0.0" ixz="0.0" iyy="1.0" iyz="0.0" izz="1.0"/>
+            <mass value="0.148495"/>
+            <inertia ixx="0.000689" ixy="0.000004" ixz="0.000012" iyy="0.000445" iyz="-0.000019" izz="0.000857"/>
         </inertial>
     </link>

File: living_lab_robot_description/urdf/head_assy.urdf.xacro (robot description, xacro)
@@ -16,7 +16,7 @@
         </collision>
         <inertial>
-            <origin xyz="0 0 0" rpy="0 0 0"/>
-            <mass value="1.0"/>
-            <inertia ixx="1.0" ixy="0.0" ixz="0.0" iyy="1.0" iyz="0.0" izz="1.0"/>
+            <origin xyz="0 0 -0.1224" rpy="0 0 0"/>
+            <mass value="6.545411"/>
+            <inertia ixx="0.085366" ixy="0.0" ixz="0.0" iyy="0.085366" iyz="0.0" izz="0.105357"/>
         </inertial>
     </link>
@@ -43,7 +43,7 @@
         </collision>
         <inertial>
-            <origin xyz="0 0 0" rpy="0 0 0"/>
-            <mass value="1.0"/>
-            <inertia ixx="1.0" ixy="0.0" ixz="0.0" iyy="1.0" iyz="0.0" izz="1.0"/>
+            <origin xyz="0.014478 0.0 -0.045490" rpy="0 0 0"/>
+            <mass value="0.186690"/>
+            <inertia ixx="0.000811" ixy="0.0" ixz="0.000012" iyy="0.000271" iyz="0.0" izz="0.000576"/>
         </inertial>
     </link>
@@ -70,7 +70,7 @@
         </collision>
         <inertial>
-            <origin xyz="0 0 0" rpy="0 0 0"/>
-            <mass value="5.0"/>
-            <inertia ixx="1.0" ixy="0.0" ixz="0.0" iyy="1.0" iyz="0.0" izz="1.0"/>
+            <origin xyz="-0.098000 0 0.057616" rpy="0 0 0"/>
+            <mass value="2.540090"/>
+            <inertia ixx="0.022353" ixy="0.0" ixz="0.0" iyy="0.022353" iyz="0.0" izz="0.040886"/>
         </inertial>
     </link>
@@ -88,9 +88,9 @@
     <xacro:insert_rgbd_camera_sensor name="camera"/>
     <link name="gaze_link">
-        <inertial>
+        <!-- <inertial>
             <origin xyz="0 0 0" rpy="0 0 0"/>
-            <mass value="1.0"/>
-            <inertia ixx="1.0" ixy="0.0" ixz="0.0" iyy="1.0" iyz="0.0" izz="1.0"/>
-        </inertial>
+            <mass value="0.01"/>
+            <inertia ixx="0.0001" ixy="0.0" ixz="0.0" iyy="0.0001" iyz="0.0" izz="0.0001"/>
+        </inertial> -->
     </link>
     <joint name="gaze_fixed_joint" type="fixed">

File: living_lab_robot_description/urdf/mobile_assy.urdf.xacro (robot description, xacro)
@@ -16,7 +16,7 @@
         </collision>
         <inertial>
-            <origin xyz="0 0 0" rpy="0 0 0"/>
+            <origin xyz="0 0 0.1111" rpy="0 0 0"/>
             <mass value="30.0"/>
-            <inertia ixx="10.0" ixy="0.0" ixz="0.0" iyy="10.0" iyz="0.0" izz="10.0"/>
+            <inertia ixx="0.9808" ixy="0.0" ixz="0.0" iyy="0.9808" iyz="0.0" izz="1.5024"/>
         </inertial>
     </link>
@@ -27,9 +27,9 @@
     </joint>
     <link name="front_hokuyo_link">
-        <inertial>
+        <!-- <inertial>
             <origin xyz="0 0 0" rpy="0 0 0"/>
             <mass value="1.0"/>
             <inertia ixx="1.0" ixy="0.0" ixz="0.0" iyy="1.0" iyz="0.0" izz="1.0"/>
-        </inertial>
+        </inertial> -->
     </link>
     <xacro:insert_hokuyo_sensor name="front" />
@@ -40,9 +40,9 @@
     </joint>
     <link name="rear_hokuyo_link">
-        <inertial>
+        <!-- <inertial>
             <origin xyz="0 0 0" rpy="0 0 0"/>
             <mass value="1.0"/>
             <inertia ixx="1.0" ixy="0.0" ixz="0.0" iyy="1.0" iyz="0.0" izz="1.0"/>
-        </inertial>
+        </inertial> -->
     </link>
     <xacro:insert_hokuyo_sensor name="rear" />
@@ -60,13 +60,13 @@
         </visual>
         <collision>
-            <origin xyz="0 0 0" rpy="0 0 0"/>
+            <origin xyz="0 0 0" rpy="${pi/2} 0 0"/>
             <geometry>
-                <mesh filename="package://living_lab_robot_description/meshes/omni_wheel.dae" scale="1 1 1"/>
+                <cylinder radius="0.065" length="0.06"/>
             </geometry>
         </collision>
         <inertial>
-            <origin xyz="0 0 0" rpy="0 0 0"/>
-            <mass value="1.0"/>
-            <inertia ixx="1.0" ixy="0.0" ixz="0.0" iyy="1.0" iyz="0.0" izz="1.0"/>
+            <origin xyz="0 -0.0015 0" rpy="0 0 0"/>
+            <mass value="0.2"/>
+            <inertia ixx="0.000324" ixy="0.0" ixz="0.0" iyy="0.000510" iyz="0.0" izz="0.000324"/>
         </inertial>
     </link>
@@ -86,13 +86,13 @@
         </visual>
         <collision>
-            <origin xyz="0 0 0" rpy="0 0 0"/>
+            <origin xyz="0 0 0" rpy="${pi/2} 0 0"/>
             <geometry>
-                <mesh filename="package://living_lab_robot_description/meshes/omni_wheel.dae" scale="1 1 1"/>
+                <cylinder radius="0.065" length="0.06"/>
             </geometry>
         </collision>
         <inertial>
-            <origin xyz="0 0 0" rpy="0 0 0"/>
-            <mass value="1.0"/>
-            <inertia ixx="1.0" ixy="0.0" ixz="0.0" iyy="1.0" iyz="0.0" izz="1.0"/>
+            <origin xyz="0 -0.0015 0" rpy="0 0 0"/>
+            <mass value="0.2"/>
+            <inertia ixx="0.000324" ixy="0.0" ixz="0.0" iyy="0.000510" iyz="0.0" izz="0.000324"/>
         </inertial>
     </link>
@@ -112,13 +112,13 @@
         </visual>
         <collision>
-            <origin xyz="0 0 0" rpy="0 0 0"/>
+            <origin xyz="0 0 0" rpy="${pi/2} 0 0"/>
             <geometry>
-                <mesh filename="package://living_lab_robot_description/meshes/omni_wheel.dae" scale="1 1 1"/>
+                <cylinder radius="0.065" length="0.06"/>
             </geometry>
         </collision>
         <inertial>
-            <origin xyz="0 0 0" rpy="0 0 0"/>
-            <mass value="1.0"/>
-            <inertia ixx="1.0" ixy="0.0" ixz="0.0" iyy="1.0" iyz="0.0" izz="1.0"/>
+            <origin xyz="0 -0.0015 0" rpy="0 0 0"/>
+            <mass value="0.2"/>
+            <inertia ixx="0.000324" ixy="0.0" ixz="0.0" iyy="0.000510" iyz="0.0" izz="0.000324"/>
         </inertial>
     </link>

File: living_lab_robot_description/urdf/robot.urdf.xacro (robot description, xacro)
@@ -5,6 +5,7 @@
     <xacro:include filename="$(find living_lab_robot_description)/urdf/mobile_assy.urdf.xacro"/>
     <xacro:include filename="$(find living_lab_robot_description)/urdf/body_assy.urdf.xacro"/>
+    <!--
     <xacro:include filename="$(find living_lab_robot_description)/urdf/arm.urdf.xacro"/>
-    <xacro:include filename="$(find living_lab_robot_description)/urdf/gripper.urdf.xacro"/>
+    <xacro:include filename="$(find living_lab_robot_description)/urdf/gripper.urdf.xacro"/>-->
     <xacro:include filename="$(find living_lab_robot_description)/urdf/head_assy.urdf.xacro"/>
 </robot>
