Commit message: Bug fixed for demo

File: living_lab_robot_description/urdf/arm.urdf.xacro (robot description, xacro)
@@ -25,5 +25,5 @@
         <origin xyz="0.035 0 -0.0228" rpy="0 0 0"/>
         <axis xyz="1 0 0"/>
-        <limit lower="-0.15" upper="0" velocity="1.0" effort="1000"/>
+        <limit lower="0" upper="0" velocity="1.0" effort="1000"/>
     </joint>
     <xacro:insert_position_transmission name="arm_base_joint" />

Commit message: Use joint_state_publisher_gui
Change the limits of arm_base_joint

File: living_lab_robot_description/urdf/arm.urdf.xacro (robot description, xacro)
@@ -25,5 +25,5 @@
         <origin xyz="0.035 0 -0.0228" rpy="0 0 0"/>
         <axis xyz="1 0 0"/>
-        <limit lower="0" upper="0" velocity="1.0" effort="1000"/>
+        <limit lower="-0.15" upper="0" velocity="1.0" effort="1000"/>
     </joint>
     <xacro:insert_position_transmission name="arm_base_joint" />

Commit message: Adjust the physical values

File: living_lab_robot_description/urdf/arm.urdf.xacro (robot description, xacro)
@@ -15,7 +15,7 @@
         </collision>
         <inertial>
-            <origin xyz="0 0 0" rpy="0 0 0"/>
-            <mass value="1.0"/>
-            <inertia ixx="1.0" ixy="0.0" ixz="0.0" iyy="1.0" iyz="0.0" izz="1.0"/>
+            <origin xyz="0.0791 0 -0.0397" rpy="0 0 0"/>
+            <mass value="0.25"/>
+            <inertia ixx="0.000190" ixy="0.0" ixz="0.0" iyy="0.000508" iyz="0.0" izz="0.000434"/>
         </inertial>
     </link>
@@ -42,7 +42,7 @@
         </collision>
         <inertial>
-            <origin xyz="0 0 0" rpy="0 0 0"/>
-            <mass value="1.0"/>
-            <inertia ixx="1.0" ixy="0.0" ixz="0.0" iyy="1.0" iyz="0.0" izz="1.0"/>
+            <origin xyz="0.0333 0 0" rpy="0 0 0"/>
+            <mass value="0.39"/>
+            <inertia ixx="0.000954" ixy="0.0" ixz="0.0" iyy="0.000283" iyz="0.0" izz="0.000954"/>
         </inertial>
     </link>
@@ -69,7 +69,7 @@
         </collision>
         <inertial>
-            <origin xyz="0 0 0" rpy="0 0 0"/>
-            <mass value="1.0"/>
-            <inertia ixx="1.0" ixy="0.0" ixz="0.0" iyy="1.0" iyz="0.0" izz="1.0"/>
+            <origin xyz="0.1691 0 0.0089" rpy="0 0 0"/>
+            <mass value="0.12"/>
+            <inertia ixx="0.004171" ixy="0.0" ixz="-0.001476" iyy="0.014517" iyz="0.0" izz="0.016818"/>
         </inertial>
     </link>
@@ -96,7 +96,7 @@
         </collision>
         <inertial>
-            <origin xyz="0 0 0" rpy="0 0 0"/>
-            <mass value="1.0"/>
-            <inertia ixx="1.0" ixy="0.0" ixz="0.0" iyy="1.0" iyz="0.0" izz="1.0"/>
+            <origin xyz="0.1137 0 -0.0419" rpy="0 0 0"/>
+            <mass value="0.14"/>
+            <inertia ixx="0.000363" ixy="0.000002" ixz="-0.000009" iyy="0.000832" iyz="0.0" izz="0.001036"/>
         </inertial>
     </link>
@@ -123,7 +123,7 @@
         </collision>
         <inertial>
-            <origin xyz="0 0 0" rpy="0 0 0"/>
-            <mass value="1.0"/>
-            <inertia ixx="1.0" ixy="0.0" ixz="0.0" iyy="1.0" iyz="0.0" izz="1.0"/>
+            <origin xyz="0.0274 0.0 0.0" rpy="0 0 0"/>
+            <mass value="0.20"/>
+            <inertia ixx="0.000315" ixy="0.0" ixz="0.0" iyy="0.000096" iyz="0.0" izz="0.000315"/>
         </inertial>
     </link>
@@ -150,7 +150,7 @@
         </collision>
         <inertial>
-            <origin xyz="0 0 0" rpy="0 0 0"/>
-            <mass value="1.0"/>
-            <inertia ixx="1.0" ixy="0.0" ixz="0.0" iyy="1.0" iyz="0.0" izz="1.0"/>
+            <origin xyz="0.0608 0 0" rpy="0 0 0"/>
+            <mass value="0.15"/>
+            <inertia ixx="0.000427" ixy="0.0" ixz="0.0" iyy="0.000507" iyz="0.0" izz="0.000774"/>
         </inertial>
     </link>
@@ -162,10 +162,10 @@
         <limit lower="${-95/180*pi}" upper="${95/180*pi}" velocity="0.4" effort="1000"/>
     </joint>
-    <xacro:insert_position_transmission name="arm5_joint" />
+    <xacro:insert_position_transmission name="arm5_joint" /> -->
     <link name="arm_link6">
         <inertial>
             <origin xyz="0 0 0" rpy="0 0 0"/>
-            <mass value="1.0"/>
-            <inertia ixx="1.0" ixy="0.0" ixz="0.0" iyy="1.0" iyz="0.0" izz="1.0"/>
+            <mass value="0.00001"/>
+            <inertia ixx="0.00001" ixy="0.0" ixz="0.0" iyy="0.00001" iyz="0.0" izz="0.00001"/>
         </inertial>
     </link>

File: living_lab_robot_description/urdf/body_assy.urdf.xacro (robot description, xacro)
@@ -16,6 +16,6 @@
         <inertial>
             <origin xyz="0 0 0.3780" rpy="0 0 0"/>
-            <mass value="5.0"/>
-            <inertia ixx="0.278381" ixy="0.0" ixz="0.0" iyy="0.278381" iyz="0.0" izz="0.080481"/>
+            <mass value="3.21"/>
+            <inertia ixx="0.263797" ixy="0.000014" ixz="-0.000365" iyy="0.255334" iyz="-0.000303" izz="0.069846"/>
         </inertial>
     </link>
@@ -43,6 +43,6 @@
         <inertial>
             <origin xyz="0 0 0" rpy="0 0 0"/>
-            <mass value="0.148495"/>
-            <inertia ixx="0.000689" ixy="0.000004" ixz="0.000012" iyy="0.000445" iyz="-0.000019" izz="0.000857"/>
+            <mass value="0.31"/>
+            <inertia ixx="0.001422" ixy="0.000007" ixz="0.000024" iyy="0.000917" iyz="-0.000039" izz="0.001769"/>
         </inertial>
     </link>

File: living_lab_robot_description/urdf/mobile_assy.urdf.xacro (robot description, xacro)
@@ -17,6 +17,6 @@
         <inertial>
             <origin xyz="0 0 0.1111" rpy="0 0 0"/>
-            <mass value="30.0"/>
-            <inertia ixx="0.9808" ixy="0.0" ixz="0.0" iyy="0.9808" iyz="0.0" izz="1.5024"/>
+            <mass value="52.01"/>
+            <inertia ixx="1.700489" ixy="0.0" ixz="0.0" iyy="1.700489" iyz="0.0" izz="2.604803"/>
         </inertial>
     </link>
@@ -67,6 +67,6 @@
         <inertial>
             <origin xyz="0 -0.0015 0" rpy="0 0 0"/>
-            <mass value="0.2"/>
-            <inertia ixx="0.000324" ixy="0.0" ixz="0.0" iyy="0.000510" iyz="0.0" izz="0.000324"/>
+            <mass value="0.42"/>
+            <inertia ixx="0.000562" ixy="0.0" ixz="0.0" iyy="0.000884" iyz="0.0" izz="0.000562"/>
         </inertial>
     </link>
@@ -93,6 +93,6 @@
         <inertial>
             <origin xyz="0 -0.0015 0" rpy="0 0 0"/>
-            <mass value="0.2"/>
-            <inertia ixx="0.000324" ixy="0.0" ixz="0.0" iyy="0.000510" iyz="0.0" izz="0.000324"/>
+            <mass value="0.42"/>
+            <inertia ixx="0.000562" ixy="0.0" ixz="0.0" iyy="0.000884" iyz="0.0" izz="0.000562"/>
         </inertial>
     </link>
@@ -119,6 +119,6 @@
         <inertial>
             <origin xyz="0 -0.0015 0" rpy="0 0 0"/>
-            <mass value="0.2"/>
-            <inertia ixx="0.000324" ixy="0.0" ixz="0.0" iyy="0.000510" iyz="0.0" izz="0.000324"/>
+            <mass value="0.42"/>
+            <inertia ixx="0.000562" ixy="0.0" ixz="0.0" iyy="0.000884" iyz="0.0" izz="0.000562"/>
         </inertial>
     </link>

File: living_lab_robot_description/urdf/robot.urdf.xacro (robot description, xacro)
@@ -5,7 +5,6 @@
     <xacro:include filename="$(find living_lab_robot_description)/urdf/mobile_assy.urdf.xacro"/>
     <xacro:include filename="$(find living_lab_robot_description)/urdf/body_assy.urdf.xacro"/>
-    <!--
     <xacro:include filename="$(find living_lab_robot_description)/urdf/arm.urdf.xacro"/>
-    <xacro:include filename="$(find living_lab_robot_description)/urdf/gripper.urdf.xacro"/>-->
-    <xacro:include filename="$(find living_lab_robot_description)/urdf/head_assy.urdf.xacro"/>
+    <!--<xacro:include filename="$(find living_lab_robot_description)/urdf/gripper.urdf.xacro"/>
+    <xacro:include filename="$(find living_lab_robot_description)/urdf/head_assy.urdf.xacro"/>-->
 </robot>
