Commit message: Sperate the link for arm_link5 and arm_link6
Add gripper which is available to control

Adjust physical values for all links

File: living_lab_robot_description/urdf/arm.urdf.xacro (robot description, xacro)
@@ -15,7 +15,7 @@
         </collision>
         <inertial>
-            <origin xyz="0.0791 0 -0.0397" rpy="0 0 0"/>
-            <mass value="0.25"/>
-            <inertia ixx="0.000190" ixy="0.0" ixz="0.0" iyy="0.000508" iyz="0.0" izz="0.000434"/>
+            <origin xyz="0.0784 0 -0.0345" rpy="0 0 0"/>
+            <mass value="0.4997"/>
+            <inertia ixx="0.000431" ixy="0.0" ixz="0.0" iyy="0.001305" iyz="0.0" izz="0.001120"/>
         </inertial>
     </link>
@@ -25,5 +25,5 @@
         <origin xyz="0.035 0 -0.0228" rpy="0 0 0"/>
         <axis xyz="1 0 0"/>
-        <limit lower="-0.15" upper="0" velocity="1.0" effort="1000"/>
+        <limit lower="-0.15" upper="0" velocity="1.0" effort="20"/>
     </joint>
     <xacro:insert_position_transmission name="arm_base_joint" />
@@ -42,7 +42,7 @@
         </collision>
         <inertial>
-            <origin xyz="0.0333 0 0" rpy="0 0 0"/>
-            <mass value="0.39"/>
-            <inertia ixx="0.000954" ixy="0.0" ixz="0.0" iyy="0.000283" iyz="0.0" izz="0.000954"/>
+            <origin xyz="0.0330 0 0" rpy="0 0 0"/>
+            <mass value="0.5067"/>
+            <inertia ixx="0.001238" ixy="0.0" ixz="0.0" iyy="0.000376" iyz="0.0" izz="0.001238"/>
         </inertial>
     </link>
@@ -52,5 +52,5 @@
         <origin xyz="0.15612 0 -0.051215" rpy="0 0 0"/>
         <axis xyz="1 0 0"/>
-        <limit lower="${-180/180*pi}" upper="${180/180*pi}" velocity="0.4" effort="1000"/>
+        <limit lower="${-180/180*pi}" upper="${180/180*pi}" velocity="0.4" effort="20"/>
     </joint>
     <xacro:insert_position_transmission name="arm1_joint" />
@@ -69,7 +69,7 @@
         </collision>
         <inertial>
-            <origin xyz="0.1691 0 0.0089" rpy="0 0 0"/>
-            <mass value="0.12"/>
-            <inertia ixx="0.004171" ixy="0.0" ixz="-0.001476" iyy="0.014517" iyz="0.0" izz="0.016818"/>
+            <origin xyz="0.1642 0 0.0083" rpy="0 0 0"/>
+            <mass value="1.1597"/>
+            <inertia ixx="0.005197" ixy="0" ixz="-0.001920" iyy="0.017977" iyz="0" izz="0.020790"/>
         </inertial>
     </link>
@@ -79,5 +79,5 @@
         <origin xyz="0.033 0 0" rpy="0 0 0"/>
         <axis xyz="0 1 0"/>
-        <limit lower="${-95/180*pi}" upper="${95/180*pi}" velocity="0.4" effort="1000"/>
+        <limit lower="${-95/180*pi}" upper="${95/180*pi}" velocity="0.4" effort="20"/>
     </joint>
     <xacro:insert_position_transmission name="arm2_joint" />
@@ -96,7 +96,7 @@
         </collision>
         <inertial>
-            <origin xyz="0.1137 0 -0.0419" rpy="0 0 0"/>
-            <mass value="0.14"/>
-            <inertia ixx="0.000363" ixy="0.000002" ixz="-0.000009" iyy="0.000832" iyz="0.0" izz="0.001036"/>
+            <origin xyz="0.1137 0 -0.0409" rpy="0 0 0"/>
+            <mass value="1.1757"/>
+            <inertia ixx="0.001933" ixy="0" ixz="0" iyy="0.005040" iyz="0.0" izz="0.006220"/>
         </inertial>
     </link>
@@ -106,5 +106,5 @@
         <origin xyz="0.264 0 0.030" rpy="0 0 0"/>
         <axis xyz="0 1 0"/>
-        <limit lower="${-180/180*pi}" upper="${5/180*pi}" velocity="0.4" effort="1000"/>
+        <limit lower="${-180/180*pi}" upper="${5/180*pi}" velocity="0.4" effort="20"/>
     </joint>
     <xacro:insert_position_transmission name="arm3_joint" />
@@ -123,7 +123,7 @@
         </collision>
         <inertial>
-            <origin xyz="0.0274 0.0 0.0" rpy="0 0 0"/>
-            <mass value="0.20"/>
-            <inertia ixx="0.000315" ixy="0.0" ixz="0.0" iyy="0.000096" iyz="0.0" izz="0.000315"/>
+            <origin xyz="0.0269 0.0 0.0" rpy="0 0 0"/>
+            <mass value="0.2697"/>
+            <inertia ixx="0.000422" ixy="0.0" ixz="0.0" iyy="0.000133" iyz="0.0" izz="0.000422"/>
         </inertial>
     </link>
@@ -133,5 +133,5 @@
         <origin xyz="0.231 0 -0.042" rpy="0 0 0"/>
         <axis xyz="1 0 0"/>
-        <limit lower="${-180/180*pi}" upper="${180/180*pi}" velocity="0.4" effort="1000"/>
+        <limit lower="${-180/180*pi}" upper="${180/180*pi}" velocity="0.4" effort="20"/>
     </joint>
     <xacro:insert_position_transmission name="arm4_joint" />
@@ -150,7 +150,7 @@
         </collision>
         <inertial>
-            <origin xyz="0.0608 0 0" rpy="0 0 0"/>
-            <mass value="0.15"/>
-            <inertia ixx="0.000427" ixy="0.0" ixz="0.0" iyy="0.000507" iyz="0.0" izz="0.000774"/>
+            <origin xyz="0.0667 0 -0.0005" rpy="0 0 0"/>
+            <mass value="0.3885"/>
+            <inertia ixx="0.000462" ixy="0.0" ixz="0.0" iyy="0.000460" iyz="0.0" izz="0.000781"/>
         </inertial>
     </link>
@@ -160,12 +160,24 @@
         <origin xyz="0.027 0 0" rpy="0 0 0"/>
         <axis xyz="0 1 0"/>
-        <limit lower="${-95/180*pi}" upper="${95/180*pi}" velocity="0.4" effort="1000"/>
+        <limit lower="${-95/180*pi}" upper="${95/180*pi}" velocity="0.4" effort="20"/>
     </joint>
-    <xacro:insert_position_transmission name="arm5_joint" /> -->
+    <xacro:insert_position_transmission name="arm5_joint" />
     <link name="arm_link6">
+        <visual>
+            <origin xyz="0 0 0" rpy="0 0 0"/>
+            <geometry>
+                <mesh filename="package://living_lab_robot_description/meshes/arm_link6.dae" scale="1 1 1"/>
+            </geometry>
+        </visual>
+        <collision>
+            <origin xyz="0 0 0" rpy="0 0 0"/>
+            <geometry>
+                <mesh filename="package://living_lab_robot_description/meshes/arm_link6.dae" scale="1 1 1"/>
+            </geometry>
+        </collision>
         <inertial>
-            <origin xyz="0 0 0" rpy="0 0 0"/>
-            <mass value="0.00001"/>
-            <inertia ixx="0.00001" ixy="0.0" ixz="0.0" iyy="0.00001" iyz="0.0" izz="0.00001"/>
+            <origin xyz="-0.0030 0 0" rpy="0 0 0"/>
+            <mass value="0.0038"/>
+            <inertia ixx="0.0000006" ixy="0.0" ixz="0.0" iyy="0.0000003" iyz="0.0" izz="0.0000003"/>
         </inertial>
     </link>
@@ -175,5 +187,5 @@
         <origin xyz="0.123 0 0" rpy="0 0 0"/>
         <axis xyz="1 0 0"/>
-        <limit lower="${-180/180*pi}" upper="${180/180*pi}" velocity="0.4" effort="1000"/>
+        <limit lower="${-180/180*pi}" upper="${180/180*pi}" velocity="0.4" effort="20"/>
     </joint>
     <xacro:insert_position_transmission name="arm6_joint" />

File: living_lab_robot_description/urdf/gazebo.urdf.xacro (robot description, xacro)
@@ -12,8 +12,30 @@
             <odometryTopic>odom</odometryTopic>
             <odometryFrame>odom</odometryFrame>
-            <odometryRate>30.0</odometryRate>
-            <robotBaseFrame>base_footprint</robotBaseFrame>
+            <odometryRate>50.0</odometryRate>
+            <robotBaseFrame>base_link</robotBaseFrame>
         </plugin>
     </gazebo>
+    <gazebo reference="omni_wheel_1">
+        <mu1 value="0.0"/>
+        <mu1 value="0.0"/>
+    </gazebo>
+    <gazebo reference="omni_wheel_2">
+        <mu1 value="0.0"/>
+        <mu1 value="0.0"/>
+    </gazebo>
+    <gazebo reference="omni_wheel_3">
+        <mu1 value="0.0"/>
+        <mu1 value="0.0"/>
+    </gazebo>
+    <xacro:macro name="insert_mimic_joint" params="reference name multiplier offset">
+        <gazebo>
+            <plugin name="mimic_${name}" filename="libgazebo_mimic_joint_plugin.so">
+                <joint>${reference}</joint>
+                <mimicJoint>${name}</mimicJoint>
+                <multiplier>${multiplier}</multiplier>
+                <offset>${offset}</offset>
+            </plugin>
+        </gazebo>
+    </xacro:macro>
     <gazebo reference="base_link">
         <mu1 value="0.0"/>

File: living_lab_robot_description/urdf/gripper.urdf.xacro (robot description, xacro)
@@ -1,17 +1,207 @@
 <?xml version="1.0"?>
-<robot xmlns:xacro="http://www.ros.org/wiki/xacro">
-    <link name="gripper">
-        <visual>
+<robot name="robotis_gripper" xmlns:xacro="http://ros.org/wiki/xacro">
+    <xacro:macro name="robotis_gripper" params="parent *origin prefix:=''">
+        <link name="gripper_base_link">
+            <visual>
+                <origin xyz="0 0 0" rpy="0 0 0"/>
+                <geometry>
+                    <mesh filename="package://robotis_gripper_description/meshes/gripper_base.dae" scale="1 1 1"/>
+                </geometry>
+            </visual>
+            <collision>
+                <origin xyz="0 0 0" rpy="0 0 0"/>
+                <geometry>
+                    <mesh filename="package://robotis_gripper_description/meshes/gripper_base.dae" scale="1 1 1"/>
+                </geometry>
+            </collision>
+            <inertial>
+                <origin xyz="0.03022 0.0 0.00109" rpy="0 0 0"/>
+                <mass value="0.3910"/>
+                <inertia ixx="0.000276" ixy="0.0" ixz="0.0" iyy="0.000198" iyz="0.0" izz="0.000265"/>
+            </inertial>
+        </link>
+        <joint name="gripper_base_fixed_joint" type="fixed">
+            <parent link="${parent}"/>
+            <child link="gripper_base_link"/>
             <origin xyz="0 0 0" rpy="0 0 0"/>
-            <geometry>
-                <mesh filename="package://living_lab_robot_description/meshes/gripper.dae" scale="1 1 1"/>
-            </geometry>
-        </visual>
-        <collision>
-            <origin xyz="0 0 0" rpy="0 0 0"/>
-            <geometry>
-                <mesh filename="package://living_lab_robot_description/meshes/gripper.dae" scale="1 1 1"/>
-            </geometry>
-        </collision>
+        </joint>
+        <link name="gripper_l_inner_link">
+            <visual>
+                <origin xyz="0 0 0" rpy="0 0 0"/>
+                <geometry>
+                    <mesh filename="package://robotis_gripper_description/meshes/inner_link.dae" scale="1 1 1"/>
+                </geometry>
+            </visual>
+            <collision>
+                <origin xyz="0 0 0" rpy="0 0 0"/>
+                <geometry>
+                    <mesh filename="package://robotis_gripper_description/meshes/inner_link.dae" scale="1 1 1"/>
+                </geometry>
+            </collision>
+            <inertial>
+                <origin xyz="0.02966 -0.00035 0.00002" rpy="0 0 0"/>
+                <mass value="0.0158"/>
+                <inertia ixx="0.000002" ixy="0.0" ixz="0.0" iyy="0.000006" iyz="0.0" izz="0.000004"/>
+            </inertial>
+        </link>
+        <joint name="gripper_joint" type="revolute">
+            <parent link="gripper_base_link"/>
+            <child link="gripper_l_inner_link"/>
+            <origin xyz="0.048 0.008 0" rpy="0 0 0"/>
+            <axis xyz="0 0 1"/>
+            <limit effort="1000" velocity="1.0" lower="-0.075" upper="1.2217"/>
+        </joint>
+        <transmission name="gripper_joint_tran">
+            <type>transmission_interface/SimpleTransmission</type>
+            <joint name="gripper_joint" >
+                <hardwareInterface>hardware_interface/PositionJointInterface</hardwareInterface>
+                <mechanicalReduction>1</mechanicalReduction>
+            </joint>
+            <actuator name="gripper_joint_motor">
+                <hardwareInterface>hardware_interface/PositionJointInterface</hardwareInterface>
+                <mechanicalReduction>1</mechanicalReduction>
+            </actuator>
+        </transmission>
+        <link name="gripper_r_inner_link">
+            <visual>
+                <origin xyz="0 0 0" rpy="${pi} 0 0"/>
+                <geometry>
+                    <mesh filename="package://robotis_gripper_description/meshes/inner_link.dae" scale="1 1 1"/>
+                </geometry>
+            </visual>
+            <collision>
+                <origin xyz="0 0 0" rpy="${pi} 0 0"/>
+                <geometry>
+                    <mesh filename="package://robotis_gripper_description/meshes/inner_link.dae" scale="1 1 1"/>
+                </geometry>
+            </collision>
+            <inertial>
+                <origin xyz="0.02966 -0.00035 0.00002" rpy="${pi} 0 0"/>
+                <mass value="0.0158"/>
+                <inertia ixx="0.000002" ixy="0.0" ixz="0.0" iyy="0.000006" iyz="0.0" izz="0.000004"/>
+            </inertial>
+        </link>
+        <joint name="gripper_r_inner_joint" type="revolute">
+            <parent link="gripper_base_link"/>
+            <child link="gripper_r_inner_link"/>
+            <origin xyz="0.048 -0.008 0" rpy="0 0 0"/>
+            <axis xyz="0 0 1"/>
+            <limit effort="1000" velocity="1.0" lower="-1.5707" upper="1.5707"/>
+            <mimic joint="gripper_joint" multiplier="-1" offset="0"/>
+        </joint>
+        <xacro:insert_mimic_joint reference="gripper_joint" name="gripper_r_inner_joint" multiplier="-1.0" offset="0.0"/>
+        <link name="gripper_l_outer_link">
+            <visual>
+                <origin xyz="0 0 0" rpy="0 0 0"/>
+                <geometry>
+                    <mesh filename="package://robotis_gripper_description/meshes/l_outer_link.dae" scale="1 1 1"/>
+                </geometry>
+            </visual>
+            <collision>
+                <origin xyz="0 0 0" rpy="0 0 0"/>
+                <geometry>
+                    <mesh filename="package://robotis_gripper_description/meshes/l_outer_link.dae" scale="1 1 1"/>
+                </geometry>
+            </collision>
+            <inertial>
+                <origin xyz="0.01616 0.02092 0.00067" rpy="0 0 0"/>
+                <mass value="0.0130"/>
+                <inertia ixx="0.000001" ixy="-0.000001" ixz="0.0" iyy="0.000006" iyz="0.0" izz="0.000006"/>
+            </inertial>
+        </link>
+        <joint name="gripper_l_outer_joint" type="revolute">
+            <parent link="gripper_base_link"/>
+            <child link="gripper_l_outer_link"/>
+            <origin xyz="0.0374 0.0186 0" rpy="0 0 0"/>
+            <axis xyz="0 0 1"/>
+            <limit effort="1000" velocity="1.0" lower="-1.5707" upper="1.5707"/>
+            <mimic joint="gripper_joint" multiplier="1" offset="-0.405"/>
+        </joint>
+        <xacro:insert_mimic_joint reference="gripper_joint" name="gripper_l_outer_joint" multiplier="1.0" offset="-0.405"/>
+        <link name="gripper_r_outer_link">
+            <visual>
+                <origin xyz="0 0 0" rpy="0 0 0"/>
+                <geometry>
+                    <mesh filename="package://robotis_gripper_description/meshes/r_outer_link.dae" scale="1 1 1"/>
+                </geometry>
+            </visual>
+            <collision>
+                <origin xyz="0 0 0" rpy="0 0 0"/>
+                <geometry>
+                    <mesh filename="package://robotis_gripper_description/meshes/r_outer_link.dae" scale="1 1 1"/>
+                </geometry>
+            </collision>
+            <inertial>
+                <origin xyz="0.01616 -0.02092 0.00065" rpy="0 0 0"/>
+                <mass value="0.0130"/>
+                <inertia ixx="0.000001" ixy="0.000001" ixz="0.0" iyy="0.000006" iyz="0.0" izz="0.000006"/>
+            </inertial>
+        </link>
+        <joint name="gripper_r_outer_joint" type="revolute">
+            <parent link="gripper_base_link"/>
+            <child link="gripper_r_outer_link"/>
+            <origin xyz="0.0374 -0.0186 0" rpy="0 0 0"/>
+            <axis xyz="0 0 1"/>
+            <limit effort="1000" velocity="1.0" lower="-1.5707" upper="1.5707"/>
+            <mimic joint="gripper_joint" multiplier="-1" offset="0.405"/>
+        </joint>
+        <xacro:insert_mimic_joint reference="gripper_joint" name="gripper_r_outer_joint" multiplier="-1.0" offset="0.405"/>
+        <link name="gripper_l_finger_link">
+            <visual>
+                <origin xyz="0 0 0" rpy="0 0 0"/>
+                <geometry>
+                    <mesh filename="package://robotis_gripper_description/meshes/finger.dae" scale="1 1 1"/>
+                </geometry>
+            </visual>
+            <collision>
+                <origin xyz="0 0 0" rpy="0 0 0"/>
+                <geometry>
+                    <mesh filename="package://robotis_gripper_description/meshes/finger.dae" scale="1 1 1"/>
+                </geometry>
+            </collision>
+            <inertial>
+                <origin xyz="0.00958 0.00643 0.00000" rpy="0 0 0"/>
+                <mass value="0.0257"/>
+                <inertia ixx="0.000003" ixy="0.000002" ixz="0.0" iyy="0.000008" iyz="0.0" izz="0.000007"/>
+            </inertial>
+        </link>
+        <joint name="gripper_l_finger_joint" type="revolute">
+            <parent link="gripper_l_inner_link"/>
+            <child link="gripper_l_finger_link"/>
+            <origin xyz="0.057 0 0" rpy="0 0 0"/>
+            <axis xyz="0 0 1"/>
+            <limit effort="1000" velocity="1.0" lower="-1.5707" upper="1.5707"/>
+            <mimic joint="gripper_joint" multiplier="-1" offset="0"/>
+        </joint>
+        <xacro:insert_mimic_joint reference="gripper_joint" name="gripper_l_finger_joint" multiplier="-1.0" offset="0.0"/>
+        <link name="gripper_r_finger_link">
+            <visual>
+                <origin xyz="0 0 0" rpy="${pi} 0 0"/>
+                <geometry>
+                    <mesh filename="package://robotis_gripper_description/meshes/finger.dae" scale="1 1 1"/>
+                </geometry>
+            </visual>
+            <collision>
+                <origin xyz="0 0 0" rpy="${pi} 0 0"/>
+                <geometry>
+                    <mesh filename="package://robotis_gripper_description/meshes/finger.dae" scale="1 1 1"/>
+                </geometry>
+            </collision>
+            <inertial>
+                <origin xyz="0.00958 -0.00643 0.00000" rpy="${pi} 0 0"/>
+                <mass value="0.0257"/>
+                <inertia ixx="0.000003" ixy="0.000002" ixz="0.0" iyy="0.000008" iyz="0.0" izz="0.000007"/>
+            </inertial>
+        </link>
+        <joint name="gripper_r_finger_joint" type="revolute">
+            <parent link="gripper_r_inner_link"/>
+            <child link="gripper_r_finger_link"/>
+            <origin xyz="0.057 0 0" rpy="0 0 0"/>
+            <axis xyz="0 0 1"/>
+            <limit effort="1000" velocity="1.0" lower="-1.5707" upper="1.5707"/>
+            <mimic joint="gripper_joint" multiplier="1" offset="0"/>
+        </joint>
+        <xacro:insert_mimic_joint reference="gripper_joint" name="gripper_r_finger_joint" multiplier="1.0" offset="0.0"/>
+        <link name="end_effector">
         <inertial>
             <origin xyz="0 0 0" rpy="0 0 0"/>
@@ -19,21 +209,10 @@
             <inertia ixx="1.0" ixy="0.0" ixz="0.0" iyy="1.0" iyz="0.0" izz="1.0"/>
         </inertial>
-    </link>
-    <joint name="gripper_mount_joint" type="fixed">
-        <parent link="arm_link6"/>
-        <child link="gripper"/>
-        <origin xyz="0 0 0" rpy="0 0 0"/>
-    </joint>
-    <link name="end_effector">
-        <inertial>
-            <origin xyz="0 0 0" rpy="0 0 0"/>
-            <mass value="1.0"/>
-            <inertia ixx="1.0" ixy="0.0" ixz="0.0" iyy="1.0" iyz="0.0" izz="1.0"/>
-        </inertial>
-    </link>
-    <joint name="gripper_joint" type="fixed">
-        <parent link="gripper"/>
-        <child link="end_effector"/>
-        <origin xyz="0.096 0 0" rpy="0 0 0"/>
-    </joint>
+        </link>
+        <joint name="eef_fixed_joint" type="fixed">
+            <parent link="gripper_base_link"/>
+            <child link="end_effector"/>
+            <origin xyz="0.12 0 0" rpy="0 0 0"/>
+        </joint>
+    </xacro:macro>
 </robot>

File: living_lab_robot_description/urdf/mobile_assy.urdf.xacro (robot description, xacro)
@@ -17,5 +17,5 @@
         <inertial>
             <origin xyz="0 0 0.1111" rpy="0 0 0"/>
-            <mass value="52.01"/>
+            <mass value="55.0"/>
             <inertia ixx="1.700489" ixy="0.0" ixz="0.0" iyy="1.700489" iyz="0.0" izz="2.604803"/>
         </inertial>
@@ -62,5 +62,6 @@
             <origin xyz="0 0 0" rpy="${pi/2} 0 0"/>
             <geometry>
-                <cylinder radius="0.065" length="0.06"/>
+                <!-- <cylinder radius="0.065" length="0.06"/> -->
+                <sphere radius="0.065"/>
             </geometry>
         </collision>
@@ -88,5 +89,6 @@
             <origin xyz="0 0 0" rpy="${pi/2} 0 0"/>
             <geometry>
-                <cylinder radius="0.065" length="0.06"/>
+                <!-- <cylinder radius="0.065" length="0.06"/> -->
+                <sphere radius="0.065"/>
             </geometry>
         </collision>
@@ -114,5 +116,6 @@
             <origin xyz="0 0 0" rpy="${pi/2} 0 0"/>
             <geometry>
-                <cylinder radius="0.065" length="0.06"/>
+                <!-- <cylinder radius="0.065" length="0.06"/> -->
+                <sphere radius="0.065"/>
             </geometry>
         </collision>

File: living_lab_robot_description/urdf/robot.urdf.xacro (robot description, xacro)
@@ -6,5 +6,8 @@
     <xacro:include filename="$(find living_lab_robot_description)/urdf/body_assy.urdf.xacro"/>
     <xacro:include filename="$(find living_lab_robot_description)/urdf/arm.urdf.xacro"/>
-    <!--<xacro:include filename="$(find living_lab_robot_description)/urdf/gripper.urdf.xacro"/>
-    <xacro:include filename="$(find living_lab_robot_description)/urdf/head_assy.urdf.xacro"/>-->
+    <xacro:include filename="$(find living_lab_robot_description)/urdf/gripper.urdf.xacro"/>
+    <robotis_gripper parent="arm_link6">
+        <origin xyz="0 0 0" rpy="0 0 0"/>
+    </robotis_gripper>
+    <xacro:include filename="$(find living_lab_robot_description)/urdf/head_assy.urdf.xacro"/>
 </robot>
