Commit message: Adjust the max speed of joints

File: living_lab_robot_description/urdf/arm.urdf.xacro (robot description, xacro)
@@ -25,5 +25,5 @@
         <origin xyz="0.035 0 -0.0228" rpy="0 0 0"/>
         <axis xyz="1 0 0"/>
-        <limit lower="-0.15" upper="0" velocity="1.0" effort="20"/>
+        <limit lower="-0.15" upper="0" velocity="0.6" effort="20"/>
     </joint>
     <xacro:insert_position_transmission name="arm_base_joint" />
@@ -52,5 +52,5 @@
         <origin xyz="0.15612 0 -0.051215" rpy="0 0 0"/>
         <axis xyz="1 0 0"/>
-        <limit lower="${-180/180*pi}" upper="${180/180*pi}" velocity="0.4" effort="20"/>
+        <limit lower="${-180/180*pi}" upper="${180/180*pi}" velocity="0.8" effort="20"/>
     </joint>
     <xacro:insert_position_transmission name="arm1_joint" />
@@ -79,5 +79,5 @@
         <origin xyz="0.033 0 0" rpy="0 0 0"/>
         <axis xyz="0 1 0"/>
-        <limit lower="${-95/180*pi}" upper="${95/180*pi}" velocity="0.4" effort="20"/>
+        <limit lower="${-95/180*pi}" upper="${95/180*pi}" velocity="0.8" effort="20"/>
     </joint>
     <xacro:insert_position_transmission name="arm2_joint" />
@@ -106,5 +106,5 @@
         <origin xyz="0.264 0 0.030" rpy="0 0 0"/>
         <axis xyz="0 1 0"/>
-        <limit lower="${-180/180*pi}" upper="${5/180*pi}" velocity="0.4" effort="20"/>
+        <limit lower="${-180/180*pi}" upper="${5/180*pi}" velocity="0.8" effort="20"/>
     </joint>
     <xacro:insert_position_transmission name="arm3_joint" />
@@ -133,5 +133,5 @@
         <origin xyz="0.231 0 -0.042" rpy="0 0 0"/>
         <axis xyz="1 0 0"/>
-        <limit lower="${-180/180*pi}" upper="${180/180*pi}" velocity="0.4" effort="20"/>
+        <limit lower="${-180/180*pi}" upper="${180/180*pi}" velocity="0.8" effort="20"/>
     </joint>
     <xacro:insert_position_transmission name="arm4_joint" />
@@ -160,5 +160,5 @@
         <origin xyz="0.027 0 0" rpy="0 0 0"/>
         <axis xyz="0 1 0"/>
-        <limit lower="${-95/180*pi}" upper="${95/180*pi}" velocity="0.4" effort="20"/>
+        <limit lower="${-95/180*pi}" upper="${95/180*pi}" velocity="0.8" effort="20"/>
     </joint>
     <xacro:insert_position_transmission name="arm5_joint" />
@@ -187,5 +187,5 @@
         <origin xyz="0.123 0 0" rpy="0 0 0"/>
         <axis xyz="1 0 0"/>
-        <limit lower="${-180/180*pi}" upper="${180/180*pi}" velocity="0.4" effort="20"/>
+        <limit lower="${-180/180*pi}" upper="${180/180*pi}" velocity="0.8" effort="20"/>
     </joint>
     <xacro:insert_position_transmission name="arm6_joint" />

File: living_lab_robot_description/urdf/body_assy.urdf.xacro (robot description, xacro)
@@ -25,5 +25,5 @@
         <origin xyz="0 0 0.242" rpy="0 0 0"/>
         <axis xyz="0 0 1"/>
-        <limit lower="${-200/180*pi}" upper="${200/180*pi}" velocity="1.0" effort="1000"/>
+        <limit lower="${-200/180*pi}" upper="${200/180*pi}" velocity="0.4" effort="1000"/>
     </joint>
     <xacro:insert_position_transmission name="body_rotate_joint" />
@@ -52,5 +52,5 @@
         <origin xyz="-0.05 0 0.665" rpy="0 0 0"/>
         <axis xyz="0 0 1"/>
-        <limit lower="-0.45" upper="0" velocity="0.04" effort="1000"/>
+        <limit lower="-0.45" upper="0" velocity="0.08" effort="1000"/>
     </joint>
     <xacro:insert_position_transmission name="elevation_joint" />

File: living_lab_robot_description/urdf/gazebo.urdf.xacro (robot description, xacro)
@@ -17,12 +17,15 @@
     </gazebo>
     <gazebo reference="omni_wheel_1">
+        <selfCollide>false</selfCollide>
         <mu1 value="0.0"/>
         <mu1 value="0.0"/>
     </gazebo>
     <gazebo reference="omni_wheel_2">
+        <selfCollide>false</selfCollide>
         <mu1 value="0.0"/>
         <mu1 value="0.0"/>
     </gazebo>
     <gazebo reference="omni_wheel_3">
+        <selfCollide>false</selfCollide>
         <mu1 value="0.0"/>
         <mu1 value="0.0"/>

File: living_lab_robot_description/urdf/mobile_assy.urdf.xacro (robot description, xacro)
@@ -60,7 +60,6 @@
         </visual>
         <collision>
-            <origin xyz="0 0 0" rpy="${pi/2} 0 0"/>
+            <origin xyz="0 0 0" rpy="0 0 0"/>
             <geometry>
-                <!-- <cylinder radius="0.065" length="0.06"/> -->
                 <sphere radius="0.065"/>
             </geometry>
@@ -87,7 +86,6 @@
         </visual>
         <collision>
-            <origin xyz="0 0 0" rpy="${pi/2} 0 0"/>
+            <origin xyz="0 0 0" rpy="0 0 0"/>
             <geometry>
-                <!-- <cylinder radius="0.065" length="0.06"/> -->
                 <sphere radius="0.065"/>
             </geometry>
@@ -114,7 +112,6 @@
         </visual>
         <collision>
-            <origin xyz="0 0 0" rpy="${pi/2} 0 0"/>
+            <origin xyz="0 0 0" rpy="0 0 0"/>
             <geometry>
-                <!-- <cylinder radius="0.065" length="0.06"/> -->
                 <sphere radius="0.065"/>
             </geometry>

Commit message: Add joint constraints for moveit client

File: living_lab_robot_description/urdf/arm.urdf.xacro (robot description, xacro)
@@ -25,5 +25,5 @@
         <origin xyz="0.035 0 -0.0228" rpy="0 0 0"/>
         <axis xyz="1 0 0"/>
-        <limit lower="-0.15" upper="0" velocity="0.6" effort="20"/>
+        <limit lower="-0.15" upper="0" velocity="0.06" effort="20"/>
     </joint>
     <xacro:insert_position_transmission name="arm_base_joint" />

Commit message: Add constraints for arm_controller
Add dependencies for packages

Bug fixed

File: living_lab_robot_description/urdf/arm.urdf.xacro (robot description, xacro)
@@ -52,5 +52,5 @@
         <origin xyz="0.15612 0 -0.051215" rpy="0 0 0"/>
         <axis xyz="1 0 0"/>
-        <limit lower="${-180/180*pi}" upper="${180/180*pi}" velocity="0.8" effort="20"/>
+        <limit lower="${-180/180*pi}" upper="${180/180*pi}" velocity="1.0" effort="20"/>
     </joint>
     <xacro:insert_position_transmission name="arm1_joint" />
@@ -79,5 +79,5 @@
         <origin xyz="0.033 0 0" rpy="0 0 0"/>
         <axis xyz="0 1 0"/>
-        <limit lower="${-95/180*pi}" upper="${95/180*pi}" velocity="0.8" effort="20"/>
+        <limit lower="${-95/180*pi}" upper="${95/180*pi}" velocity="1.0" effort="20"/>
     </joint>
     <xacro:insert_position_transmission name="arm2_joint" />
@@ -106,5 +106,5 @@
         <origin xyz="0.264 0 0.030" rpy="0 0 0"/>
         <axis xyz="0 1 0"/>
-        <limit lower="${-180/180*pi}" upper="${5/180*pi}" velocity="0.8" effort="20"/>
+        <limit lower="${-180/180*pi}" upper="${5/180*pi}" velocity="1.0" effort="20"/>
     </joint>
     <xacro:insert_position_transmission name="arm3_joint" />
@@ -133,5 +133,5 @@
         <origin xyz="0.231 0 -0.042" rpy="0 0 0"/>
         <axis xyz="1 0 0"/>
-        <limit lower="${-180/180*pi}" upper="${180/180*pi}" velocity="0.8" effort="20"/>
+        <limit lower="${-180/180*pi}" upper="${180/180*pi}" velocity="1.0" effort="20"/>
     </joint>
     <xacro:insert_position_transmission name="arm4_joint" />
@@ -160,5 +160,5 @@
         <origin xyz="0.027 0 0" rpy="0 0 0"/>
         <axis xyz="0 1 0"/>
-        <limit lower="${-95/180*pi}" upper="${95/180*pi}" velocity="0.8" effort="20"/>
+        <limit lower="${-95/180*pi}" upper="${95/180*pi}" velocity="1.0" effort="20"/>
     </joint>
     <xacro:insert_position_transmission name="arm5_joint" />
@@ -187,5 +187,5 @@
         <origin xyz="0.123 0 0" rpy="0 0 0"/>
         <axis xyz="1 0 0"/>
-        <limit lower="${-180/180*pi}" upper="${180/180*pi}" velocity="0.8" effort="20"/>
+        <limit lower="${-180/180*pi}" upper="${180/180*pi}" velocity="1.0" effort="20"/>
     </joint>
     <xacro:insert_position_transmission name="arm6_joint" />

File: living_lab_robot_description/urdf/body_assy.urdf.xacro (robot description, xacro)
@@ -52,5 +52,5 @@
         <origin xyz="-0.05 0 0.665" rpy="0 0 0"/>
         <axis xyz="0 0 1"/>
-        <limit lower="-0.45" upper="0" velocity="0.08" effort="1000"/>
+        <limit lower="-0.45" upper="0" velocity="0.1" effort="100"/>
     </joint>
     <xacro:insert_position_transmission name="elevation_joint" />

File: living_lab_robot_description/urdf/gazebo.urdf.xacro (robot description, xacro)
@@ -13,5 +13,5 @@
             <odometryFrame>odom</odometryFrame>
             <odometryRate>50.0</odometryRate>
-            <robotBaseFrame>base_link</robotBaseFrame>
+            <robotBaseFrame>base_footprint</robotBaseFrame>
         </plugin>
     </gazebo>

Commit message: Add joint constraint for arm_base_joint by default (moveit bug)

File: living_lab_robot_description/urdf/arm.urdf.xacro (robot description, xacro)
@@ -16,6 +16,6 @@
         <inertial>
             <origin xyz="0.0784 0 -0.0345" rpy="0 0 0"/>
-            <mass value="0.4997"/>
-            <inertia ixx="0.000431" ixy="0.0" ixz="0.0" iyy="0.001305" iyz="0.0" izz="0.001120"/>
+            <mass value="0.9000"/>
+            <inertia ixx="0.0007768" ixy="0.0" ixz="0.0" iyy="0.0023504" iyz="0.0" izz="0.0020179"/>
         </inertial>
     </link>
@@ -25,5 +25,5 @@
         <origin xyz="0.035 0 -0.0228" rpy="0 0 0"/>
         <axis xyz="1 0 0"/>
-        <limit lower="-0.15" upper="0" velocity="0.06" effort="20"/>
+        <limit lower="-0.15" upper="0" velocity="0.06" effort="100"/>
     </joint>
     <xacro:insert_position_transmission name="arm_base_joint" />
@@ -43,6 +43,6 @@
         <inertial>
             <origin xyz="0.0330 0 0" rpy="0 0 0"/>
-            <mass value="0.5067"/>
-            <inertia ixx="0.001238" ixy="0.0" ixz="0.0" iyy="0.000376" iyz="0.0" izz="0.001238"/>
+            <mass value="0.9000"/>
+            <inertia ixx="0.0021992" ixy="0.0" ixz="0.0" iyy="0.0006670" iyz="0.0" izz="0.0021992"/>
         </inertial>
     </link>
@@ -52,5 +52,5 @@
         <origin xyz="0.15612 0 -0.051215" rpy="0 0 0"/>
         <axis xyz="1 0 0"/>
-        <limit lower="${-180/180*pi}" upper="${180/180*pi}" velocity="1.0" effort="20"/>
+        <limit lower="${-180/180*pi}" upper="${180/180*pi}" velocity="1.0" effort="100"/>
     </joint>
     <xacro:insert_position_transmission name="arm1_joint" />
@@ -70,6 +70,6 @@
         <inertial>
             <origin xyz="0.1642 0 0.0083" rpy="0 0 0"/>
-            <mass value="1.1597"/>
-            <inertia ixx="0.005197" ixy="0" ixz="-0.001920" iyy="0.017977" iyz="0" izz="0.020790"/>
+            <mass value="0.9000"/>
+            <inertia ixx="0.0021659" ixy="0" ixz="0" iyy="0.0074914" iyz="0" izz="0.0086634"/>
         </inertial>
     </link>
@@ -79,5 +79,5 @@
         <origin xyz="0.033 0 0" rpy="0 0 0"/>
         <axis xyz="0 1 0"/>
-        <limit lower="${-95/180*pi}" upper="${95/180*pi}" velocity="1.0" effort="20"/>
+        <limit lower="${-95/180*pi}" upper="${95/180*pi}" velocity="1.0" effort="100"/>
     </joint>
     <xacro:insert_position_transmission name="arm2_joint" />
@@ -97,6 +97,6 @@
         <inertial>
             <origin xyz="0.1137 0 -0.0409" rpy="0 0 0"/>
-            <mass value="1.1757"/>
-            <inertia ixx="0.001933" ixy="0" ixz="0" iyy="0.005040" iyz="0.0" izz="0.006220"/>
+            <mass value="0.8000"/>
+            <inertia ixx="0.0013151" ixy="0" ixz="0" iyy="0.0034294" iyz="0.0" izz="0.0042325"/>
         </inertial>
     </link>
@@ -106,5 +106,5 @@
         <origin xyz="0.264 0 0.030" rpy="0 0 0"/>
         <axis xyz="0 1 0"/>
-        <limit lower="${-180/180*pi}" upper="${5/180*pi}" velocity="1.0" effort="20"/>
+        <limit lower="${-180/180*pi}" upper="${5/180*pi}" velocity="1.0" effort="100"/>
     </joint>
     <xacro:insert_position_transmission name="arm3_joint" />
@@ -124,6 +124,6 @@
         <inertial>
             <origin xyz="0.0269 0.0 0.0" rpy="0 0 0"/>
-            <mass value="0.2697"/>
-            <inertia ixx="0.000422" ixy="0.0" ixz="0.0" iyy="0.000133" iyz="0.0" izz="0.000422"/>
+            <mass value="0.8000"/>
+            <inertia ixx="00.0012527" ixy="0.0" ixz="0.0" iyy="0.0003956" iyz="0.0" izz="0.0012527"/>
         </inertial>
     </link>
@@ -133,5 +133,5 @@
         <origin xyz="0.231 0 -0.042" rpy="0 0 0"/>
         <axis xyz="1 0 0"/>
-        <limit lower="${-180/180*pi}" upper="${180/180*pi}" velocity="1.0" effort="20"/>
+        <limit lower="${-180/180*pi}" upper="${180/180*pi}" velocity="1.0" effort="100"/>
     </joint>
     <xacro:insert_position_transmission name="arm4_joint" />
@@ -151,6 +151,6 @@
         <inertial>
             <origin xyz="0.0667 0 -0.0005" rpy="0 0 0"/>
-            <mass value="0.3885"/>
-            <inertia ixx="0.000462" ixy="0.0" ixz="0.0" iyy="0.000460" iyz="0.0" izz="0.000781"/>
+            <mass value="0.5000"/>
+            <inertia ixx="0.0005947" ixy="0.0" ixz="0.0" iyy="0.0005919" iyz="0.0" izz="0.0010050"/>
         </inertial>
     </link>
@@ -160,5 +160,5 @@
         <origin xyz="0.027 0 0" rpy="0 0 0"/>
         <axis xyz="0 1 0"/>
-        <limit lower="${-95/180*pi}" upper="${95/180*pi}" velocity="1.0" effort="20"/>
+        <limit lower="${-95/180*pi}" upper="${95/180*pi}" velocity="1.0" effort="100"/>
     </joint>
     <xacro:insert_position_transmission name="arm5_joint" />
@@ -178,6 +178,6 @@
         <inertial>
             <origin xyz="-0.0030 0 0" rpy="0 0 0"/>
-            <mass value="0.0038"/>
-            <inertia ixx="0.0000006" ixy="0.0" ixz="0.0" iyy="0.0000003" iyz="0.0" izz="0.0000003"/>
+            <mass value="0.2000"/>
+            <inertia ixx="0.0000301" ixy="0.0" ixz="0.0" iyy="0.0000156" iyz="0.0" izz="0.0000156"/>
         </inertial>
     </link>
@@ -187,5 +187,5 @@
         <origin xyz="0.123 0 0" rpy="0 0 0"/>
         <axis xyz="1 0 0"/>
-        <limit lower="${-180/180*pi}" upper="${180/180*pi}" velocity="1.0" effort="20"/>
+        <limit lower="${-180/180*pi}" upper="${180/180*pi}" velocity="1.0" effort="100"/>
     </joint>
     <xacro:insert_position_transmission name="arm6_joint" />

File: living_lab_robot_description/urdf/gripper.urdf.xacro (robot description, xacro)
@@ -203,11 +203,5 @@
         </joint>
         <xacro:insert_mimic_joint reference="gripper_joint" name="gripper_r_finger_joint" multiplier="1.0" offset="0.0"/>
-        <link name="end_effector">
-        <inertial>
-            <origin xyz="0 0 0" rpy="0 0 0"/>
-            <mass value="1.0"/>
-            <inertia ixx="1.0" ixy="0.0" ixz="0.0" iyy="1.0" iyz="0.0" izz="1.0"/>
-        </inertial>
-        </link>
+        <link name="end_effector"/>
         <joint name="eef_fixed_joint" type="fixed">
             <parent link="gripper_base_link"/>

Commit message: Adjust dynamics value for preventing vibration in Gazebo

File: living_lab_robot_description/urdf/arm.urdf.xacro (robot description, xacro)
@@ -25,5 +25,6 @@
         <origin xyz="0.035 0 -0.0228" rpy="0 0 0"/>
         <axis xyz="1 0 0"/>
-        <limit lower="-0.15" upper="0" velocity="0.06" effort="100"/>
+        <limit lower="-0.15" upper="0" velocity="0.06" effort="50"/>
+        <dynamics damping="0.01" friction="0.0"/>
     </joint>
     <xacro:insert_position_transmission name="arm_base_joint" />
@@ -52,5 +53,6 @@
         <origin xyz="0.15612 0 -0.051215" rpy="0 0 0"/>
         <axis xyz="1 0 0"/>
-        <limit lower="${-180/180*pi}" upper="${180/180*pi}" velocity="1.0" effort="100"/>
+        <limit lower="${-180/180*pi}" upper="${180/180*pi}" velocity="1.0" effort="50"/>
+        <dynamics damping="0.01" friction="0.0"/>
     </joint>
     <xacro:insert_position_transmission name="arm1_joint" />
@@ -79,5 +81,6 @@
         <origin xyz="0.033 0 0" rpy="0 0 0"/>
         <axis xyz="0 1 0"/>
-        <limit lower="${-95/180*pi}" upper="${95/180*pi}" velocity="1.0" effort="100"/>
+        <limit lower="${-95/180*pi}" upper="${95/180*pi}" velocity="1.0" effort="50"/>
+        <dynamics damping="0.01" friction="0.0"/>
     </joint>
     <xacro:insert_position_transmission name="arm2_joint" />
@@ -106,5 +109,6 @@
         <origin xyz="0.264 0 0.030" rpy="0 0 0"/>
         <axis xyz="0 1 0"/>
-        <limit lower="${-180/180*pi}" upper="${5/180*pi}" velocity="1.0" effort="100"/>
+        <limit lower="${-180/180*pi}" upper="${5/180*pi}" velocity="1.0" effort="50"/>
+        <dynamics damping="0.01" friction="0.0"/>
     </joint>
     <xacro:insert_position_transmission name="arm3_joint" />
@@ -133,5 +137,6 @@
         <origin xyz="0.231 0 -0.042" rpy="0 0 0"/>
         <axis xyz="1 0 0"/>
-        <limit lower="${-180/180*pi}" upper="${180/180*pi}" velocity="1.0" effort="100"/>
+        <limit lower="${-180/180*pi}" upper="${180/180*pi}" velocity="1.0" effort="50"/>
+        <dynamics damping="0.01" friction="0.0"/>
     </joint>
     <xacro:insert_position_transmission name="arm4_joint" />
@@ -160,5 +165,6 @@
         <origin xyz="0.027 0 0" rpy="0 0 0"/>
         <axis xyz="0 1 0"/>
-        <limit lower="${-95/180*pi}" upper="${95/180*pi}" velocity="1.0" effort="100"/>
+        <limit lower="${-95/180*pi}" upper="${95/180*pi}" velocity="1.0" effort="50"/>
+        <dynamics damping="0.01" friction="0.0"/>
     </joint>
     <xacro:insert_position_transmission name="arm5_joint" />
@@ -187,5 +193,6 @@
         <origin xyz="0.123 0 0" rpy="0 0 0"/>
         <axis xyz="1 0 0"/>
-        <limit lower="${-180/180*pi}" upper="${180/180*pi}" velocity="1.0" effort="100"/>
+        <limit lower="${-180/180*pi}" upper="${180/180*pi}" velocity="1.0" effort="50"/>
+        <dynamics damping="0.01" friction="0.0"/>
     </joint>
     <xacro:insert_position_transmission name="arm6_joint" />

File: living_lab_robot_description/urdf/body_assy.urdf.xacro (robot description, xacro)
@@ -44,5 +44,5 @@
             <origin xyz="0 0 0" rpy="0 0 0"/>
             <mass value="0.31"/>
-            <inertia ixx="0.001422" ixy="0.000007" ixz="0.000024" iyy="0.000917" iyz="-0.000039" izz="0.001769"/>
+            <inertia ixx="0.001422" ixy="0" ixz="0" iyy="0.000917" iyz="0" izz="0.001769"/>
         </inertial>
     </link>
@@ -53,4 +53,5 @@
         <axis xyz="0 0 1"/>
         <limit lower="-0.45" upper="0" velocity="0.1" effort="100"/>
+        <dynamics damping="0.01" friction="0.0"/>
     </joint>
     <xacro:insert_position_transmission name="elevation_joint" />

Commit message: Update urdf for simulation

File: living_lab_robot_description/urdf/arm.urdf.xacro (robot description, xacro)
@@ -16,5 +16,5 @@
         <inertial>
             <origin xyz="0.0784 0 -0.0345" rpy="0 0 0"/>
-            <mass value="0.9000"/>
+            <mass value="0.4997"/>
             <inertia ixx="0.0007768" ixy="0.0" ixz="0.0" iyy="0.0023504" iyz="0.0" izz="0.0020179"/>
         </inertial>
@@ -44,5 +44,5 @@
         <inertial>
             <origin xyz="0.0330 0 0" rpy="0 0 0"/>
-            <mass value="0.9000"/>
+            <mass value="0.5067"/>
             <inertia ixx="0.0021992" ixy="0.0" ixz="0.0" iyy="0.0006670" iyz="0.0" izz="0.0021992"/>
         </inertial>
@@ -128,5 +128,5 @@
         <inertial>
             <origin xyz="0.0269 0.0 0.0" rpy="0 0 0"/>
-            <mass value="0.8000"/>
+            <mass value="0.2697"/>
             <inertia ixx="00.0012527" ixy="0.0" ixz="0.0" iyy="0.0003956" iyz="0.0" izz="0.0012527"/>
         </inertial>
@@ -156,5 +156,5 @@
         <inertial>
             <origin xyz="0.0667 0 -0.0005" rpy="0 0 0"/>
-            <mass value="0.5000"/>
+            <mass value="0.3885"/>
             <inertia ixx="0.0005947" ixy="0.0" ixz="0.0" iyy="0.0005919" iyz="0.0" izz="0.0010050"/>
         </inertial>
@@ -184,5 +184,5 @@
         <inertial>
             <origin xyz="-0.0030 0 0" rpy="0 0 0"/>
-            <mass value="0.2000"/>
+            <mass value="0.0038"/>
             <inertia ixx="0.0000301" ixy="0.0" ixz="0.0" iyy="0.0000156" iyz="0.0" izz="0.0000156"/>
         </inertial>
